Commit message: xacro files updated to match actual hardware

File: urdf/hardware/ur/ur_3_ur10e.xacro (robot description, xacro)
@@ -3,12 +3,12 @@
   <xacro:include filename="$(find on_orbit)/urdf/hardware/ur/ur10e_macro.xacro"/>
   <xacro:ur10e_robot prefix="ur_3_" calibration_file="$(find on_orbit)/config/holo_params/ur_3_calibration.yaml"/>
-  <xacro:property name="dist_tool_to_ft_sensor" value="0.0315" />
+  <xacro:property name="dist_tool_to_ft_sensor" value="0.029" />
   <!--White Peg-->
   <!-- Will need to be updated after the print-->
-  <xacro:property name="peg_rad" value="0.01505"/>
-  <xacro:property name="peg_mass" value="0.14597807959"/>
-  <xacro:property name="peg_com" value="0.02715593628"/>
+  <xacro:property name="peg_rad" value="0.0079"/>
+  <xacro:property name="peg_mass" value="0.035"/>
+  <xacro:property name="peg_com" value="0.060"/>
   <!-- Will need to be updated after the print-->
-  <xacro:property name="ur_3_ee_length" value="0.209"/>
+  <xacro:property name="ur_3_ee_length" value="0.1558"/>
   <link name="ur_3_ee">
     <visual>

File: urdf/hardware/ur/ur_4_ur10e.xacro (robot description, xacro)
@@ -9,13 +9,6 @@
   <!--Short White Nozzle Attached to Robot 4-->
   <!-- Will need to be updated after the print-->
-  <xacro:property name="ur_4_ee_length" value="0.12477"/>
-  <xacro:property name="ur_4_ee_signed_dist_from_ee_to_goal" value="0.09017557238"/>
-  <!-- <link name="world"/> -->
-  <!-- <joint name="world_to_ur_4_base_link" type="fixed"> -->
-    <!-- <parent link="world"/> -->
-    <!-- <child link="ur_4_base_link"/> -->
-    <!--We will need to determine true orientation of each of robot as they are at an angle-->
-    <!-- <origin rpy="0 0 0" xyz="0 -0.9948543 -0.00045865"/> -->
-  <!-- </joint> -->
+  <xacro:property name="ur_4_ee_length" value="0.1194"/>
+  <xacro:property name="ur_4_ee_signed_dist_from_ee_to_goal" value="0.110"/>
   <link name="hw_goal"/>
   <joint name="ur_4_ee_to_goal" type="fixed">
