Commit message: significant work into developing HIL runner. Updated the urdfs and a few controllers to work for new urdf. because we do not have the ft sensors yet we are moving into planning so lets merge this branch and start a new one for planning devel

File: urdf/hardware/ur/hw_nozzle_geom.xacro (robot description, xacro)
@@ -1,14 +1,15 @@
 <?xml version="1.0"?>
 <robot xmlns:xacro="http://www.ros.org/wiki/xacro">
-  <xacro:property name="nozzle_length" value="0.0675" />
-  <xacro:property name="nozzle_geom_length" value="0.07671" />
-  <xacro:property name="nozzle_wall_width" value="0.003" />
-  <xacro:property name="nozzle_box_width" value="0.04" />
-  <xacro:property name="throat_outer_diameter" value="0.028" />
+  <xacro:property name="nozzle_length" value="0.4285" />
+  <xacro:property name="nozzle_geom_length" value="0.4451" />
+  <xacro:property name="nozzle_wall_width" value="0.005" />
+  <xacro:property name="nozzle_box_width" value="0.125" />
+  <xacro:property name="throat_outer_diameter" value="0.032" />
   <xacro:property name="throat_middle_diameter" value="${throat_outer_diameter - nozzle_wall_width}" />
-  <xacro:property name="entry_outer_diameter" value="0.09768" />
+  <xacro:property name="entry_outer_diameter" value="0.294" />
   <xacro:property name="entry_middle_diameter" value="${entry_outer_diameter - nozzle_wall_width}" />
+  <xacro:property name="entry_inner_rad" value="${(entry_outer_diameter - 2*nozzle_wall_width)/2}" />
   <xacro:property name="dist_from_centerline" value="${(throat_middle_diameter + entry_middle_diameter)/4}" />
-  <xacro:property name="slope_angle" value="0.49514949" />
+  <xacro:property name="slope_angle" value="0.3154949" />
   <xacro:macro name="hw_nozzle_geom" params="num theta">
     <link name="hw_nozzle_geom${num}">

File: urdf/hardware/ur/nozzle_base.xacro (robot description, xacro)
@@ -2,5 +2,5 @@
 <robot xmlns:xacro="http://www.ros.org/wiki/xacro">
   <xacro:property name="nozzle_base_fixture_length" value="0.0095" />
-  <xacro:property name="nozzle_base_fixture_diameter" value="0.06" />
+  <xacro:property name="nozzle_base_fixture_diameter" value="0.063" />
   <xacro:macro name="nozzle_base" params="">
   <link name="nozzle_base">

File: urdf/hardware/ur/ur_3_ur10e.xacro (robot description, xacro)
@@ -4,11 +4,13 @@
   <xacro:ur10e_robot prefix="ur_3_" calibration_file="$(find on_orbit)/config/holo_params/ur_3_calibration.yaml"/>
   <xacro:property name="dist_tool_to_ft_sensor" value="0.029" />
-  <!--White Peg-->
+  <!--Peg-->
+  <xacro:property name="peg_rad" value="0.0079"/>
+  <xacro:property name="peg_mass" value="0.260"/>
+  <xacro:property name="peg_com" value="0.071"/>
   <!-- Will need to be updated after the print-->
-  <xacro:property name="peg_rad" value="0.0079"/>
-  <xacro:property name="peg_mass" value="0.035"/>
-  <xacro:property name="peg_com" value="0.060"/>
-  <!-- Will need to be updated after the print-->
-  <xacro:property name="ur_3_ee_length" value="0.1558"/>
+  <!-- Old Value -->
+  <!-- <xacro:property name="ur_3_ee_length" value="0.1558"/> -->
+  <!-- New Value -->
+  <xacro:property name="ur_3_ee_length" value="0.540"/>
   <link name="ur_3_ee">
     <visual>
@@ -44,5 +46,5 @@
     <origin rpy="0 0 0" xyz="0 0 ${ur_3_ee_length}"/>
   </joint>
-  <!-- UR16 has the FT sensor-->
+  <!-- ur_3 has the FT sensor-->
   <link name="ft_sensor"/>
   <joint name="ur_3_tool0_to_ft_sensor" type="fixed">

File: urdf/hardware/ur/ur_4_ur10e.xacro (robot description, xacro)
@@ -6,9 +6,8 @@
   <xacro:include filename="$(find on_orbit)/urdf/hardware/ur/ur10e_macro.xacro"/>
   <xacro:ur10e_robot prefix="ur_4_" calibration_file="$(find on_orbit)/config/holo_params/ur_4_calibration.yaml"/>
-  <xacro:property name="dist_tool_to_ft_sensor" value="0.0315" />
   <!--Short White Nozzle Attached to Robot 4-->
   <!-- Will need to be updated after the print-->
-  <xacro:property name="ur_4_ee_length" value="0.1194"/>
-  <xacro:property name="ur_4_ee_signed_dist_from_ee_to_goal" value="0.110"/>
+  <xacro:property name="ur_4_ee_length" value="0.4785"/>
+  <xacro:property name="ur_4_ee_signed_dist_from_ee_to_goal" value="0.4656"/>
   <link name="hw_goal"/>
   <joint name="ur_4_ee_to_goal" type="fixed">

File: urdf/holodeck.urdf (robot description, URDF)
Before this commit: robot holodeck, 73 links, 72 joints
Links:
- link hw_nozzle_geom0: geometry collision box size=0.005 0.125 0.4451; visual box size=0.005 0.125 0.4451
- link hw_nozzle_geom1: geometry collision box size=0.005 0.125 0.4451; visual box size=0.005 0.125 0.4451
- link hw_nozzle_geom2: geometry collision box size=0.005 0.125 0.4451; visual box size=0.005 0.125 0.4451
- link hw_nozzle_geom3: geometry collision box size=0.005 0.125 0.4451; visual box size=0.005 0.125 0.4451
- link hw_nozzle_geom4: geometry collision box size=0.005 0.125 0.4451; visual box size=0.005 0.125 0.4451
- link hw_nozzle_geom5: geometry collision box size=0.005 0.125 0.4451; visual box size=0.005 0.125 0.4451
- link hw_nozzle_geom6: geometry collision box size=0.005 0.125 0.4451; visual box size=0.005 0.125 0.4451
- link hw_nozzle_geom7: geometry collision box size=0.005 0.125 0.4451; visual box size=0.005 0.125 0.4451
- link nozzle_base: geometry collision cylinder length=0.0095 radius=0.0315; visual cylinder length=0.0095 radius=0.0315
- link ur_3_ee: mass 0.035 -> 0.26; geometry collision cylinder length=0.54 radius=0.0079; visual cylinder length=0.54 radius=0.0079
Joints:
- joint ur_3_ee_to_peg_center: origin xyz=0 0 -0.0779 rpy=0 0 0 -> xyz=0 0 -0.27 rpy=0 0 0
- joint ur_3_tool0_to_ee: origin xyz=0 0 0.1558 rpy=0 0 0 -> xyz=0 0 0.54 rpy=0 0 0
- joint ur_4_ee_to_goal: origin xyz=0 0 0.11 rpy=0 3.141592653589793 0 -> xyz=0 0 0.4656 rpy=0 3.141592653589793 0
- joint ur_4_ee_to_hw_nozzle_geom0: origin xyz=0.029920000000000002 0.0 0.03517396538237974 rpy=0 -0.49514949 0 -> xyz=0.079 0.0 0.21311701994296112 rpy=0 -0.3154949 0
- joint ur_4_ee_to_hw_nozzle_geom1: origin xyz=0.021156634893101506 0.021156634893101503 0.03517396538237974 rpy=0 -0.49514949 0.7853981633974483 -> xyz=0.05586143571373726 0.05586143571373725 0.21311701994296112 rpy=0 -0.3154949 0.7853981633974483
- joint ur_4_ee_to_hw_nozzle_geom2: origin xyz=1.8320716115244406e-18 0.029920000000000002 0.03517396538237974 rpy=0 -0.49514949 1.5707963267948966 -> xyz=4.837354856632045e-18 0.079 0.21311701994296112 rpy=0 -0.3154949 1.5707963267948966
- joint ur_4_ee_to_hw_nozzle_geom3: origin xyz=-0.021156634893101503 0.021156634893101506 0.03517396538237974 rpy=0 -0.49514949 2.356194490192345 -> xyz=-0.05586143571373725 0.05586143571373726 0.21311701994296112 rpy=0 -0.3154949 2.356194490192345
- joint ur_4_ee_to_hw_nozzle_geom4: origin xyz=-0.029920000000000002 3.664143223048881e-18 0.03517396538237974 rpy=0 -0.49514949 3.141592653589793 -> xyz=-0.079 9.67470971326409e-18 0.21311701994296112 rpy=0 -0.3154949 3.141592653589793
- joint ur_4_ee_to_hw_nozzle_geom5: origin xyz=-0.021156634893101506 -0.021156634893101503 0.03517396538237974 rpy=0 -0.49514949 3.9269908169872414 -> xyz=-0.055861435713737265 -0.05586143571373725 0.21311701994296112 rpy=0 -0.3154949 3.9269908169872414
- joint ur_4_ee_to_hw_nozzle_geom6: origin xyz=-5.496214834573321e-18 -0.029920000000000002 0.03517396538237974 rpy=0 -0.49514949 4.71238898038469 -> xyz=-1.4512064569896134e-17 -0.079 0.21311701994296112 rpy=0 -0.3154949 4.71238898038469
- joint ur_4_ee_to_hw_nozzle_geom7: origin xyz=0.0211566348931015 -0.021156634893101506 0.03517396538237974 rpy=0 -0.49514949 5.497787143782138 -> xyz=0.055861435713737244 -0.055861435713737265 0.21311701994296112 rpy=0 -0.3154949 5.497787143782138
- joint ur_4_ee_to_tube_geom0: origin xyz=0.0127 0.0 0.08975 rpy=0 0 0 -> xyz=0.0127 0.0 0.45075 rpy=0 0 0
- joint ur_4_ee_to_tube_geom1: origin xyz=0.008980256121069154 0.008980256121069152 0.08975 rpy=0 0 0.7853981633974483 -> xyz=0.008980256121069154 0.008980256121069152 0.45075 rpy=0 0 0.7853981633974483
- joint ur_4_ee_to_tube_geom2: origin xyz=7.776507174585693e-19 0.0127 0.08975 rpy=0 0 1.5707963267948966 -> xyz=7.776507174585693e-19 0.0127 0.45075 rpy=0 0 1.5707963267948966
- joint ur_4_ee_to_tube_geom3: origin xyz=-0.008980256121069152 0.008980256121069154 0.08975 rpy=0 0 2.356194490192345 -> xyz=-0.008980256121069152 0.008980256121069154 0.45075 rpy=0 0 2.356194490192345
- joint ur_4_ee_to_tube_geom4: origin xyz=-0.0127 1.5553014349171385e-18 0.08975 rpy=0 0 3.141592653589793 -> xyz=-0.0127 1.5553014349171385e-18 0.45075 rpy=0 0 3.141592653589793
- joint ur_4_ee_to_tube_geom5: origin xyz=-0.008980256121069155 -0.008980256121069152 0.08975 rpy=0 0 3.9269908169872414 -> xyz=-0.008980256121069155 -0.008980256121069152 0.45075 rpy=0 0 3.9269908169872414
- joint ur_4_ee_to_tube_geom6: origin xyz=-2.3329521523757078e-18 -0.0127 0.08975 rpy=0 0 4.71238898038469 -> xyz=-2.3329521523757078e-18 -0.0127 0.45075 rpy=0 0 4.71238898038469
- joint ur_4_ee_to_tube_geom7: origin xyz=0.00898025612106915 -0.008980256121069155 0.08975 rpy=0 0 5.497787143782138 -> xyz=0.00898025612106915 -0.008980256121069155 0.45075 rpy=0 0 5.497787143782138
- joint ur_4_tool0_to_ee: origin xyz=0 0 0.1194 rpy=0 3.14159 0 -> xyz=0 0 0.4785 rpy=0 3.14159 0

File: urdf/on_orbit.urdf (robot description, URDF)
Before this commit: robot holodeck, 48 links, 47 joints
Links:
- link hw_nozzle_geom0: geometry collision box size=0.005 0.125 0.4451; visual box size=0.005 0.125 0.4451
- link hw_nozzle_geom1: geometry collision box size=0.005 0.125 0.4451; visual box size=0.005 0.125 0.4451
- link hw_nozzle_geom2: geometry collision box size=0.005 0.125 0.4451; visual box size=0.005 0.125 0.4451
- link hw_nozzle_geom3: geometry collision box size=0.005 0.125 0.4451; visual box size=0.005 0.125 0.4451
- link hw_nozzle_geom4: geometry collision box size=0.005 0.125 0.4451; visual box size=0.005 0.125 0.4451
- link hw_nozzle_geom5: geometry collision box size=0.005 0.125 0.4451; visual box size=0.005 0.125 0.4451
- link hw_nozzle_geom6: geometry collision box size=0.005 0.125 0.4451; visual box size=0.005 0.125 0.4451
- link hw_nozzle_geom7: geometry collision box size=0.005 0.125 0.4451; visual box size=0.005 0.125 0.4451
- link nozzle_base: geometry collision cylinder length=0.0095 radius=0.0315; visual cylinder length=0.0095 radius=0.0315
- link ur_3_ee: mass 0.14597807959 -> 0.26; geometry collision cylinder length=0.54 radius=0.0079; visual cylinder length=0.54 radius=0.0079
Joints:
- joint ur_3_ee_to_peg_center: origin xyz=0 0 -0.1045 rpy=0 0 0 -> xyz=0 0 -0.27 rpy=0 0 0
- joint ur_3_tool0_to_ee: origin xyz=0 0 0.209 rpy=0 0 0 -> xyz=0 0 0.54 rpy=0 0 0
- joint ur_3_tool0_to_ft_sensor: origin xyz=0 0 0.0315 rpy=0 0 -0.53996123733 -> xyz=0 0 0.029 rpy=0 0 -0.53996123733
- joint ur_4_ee_to_goal: origin xyz=0 0 0.09017557238 rpy=0 3.141592653589793 0 -> xyz=0 0 0.4656 rpy=0 3.141592653589793 0
- joint ur_4_ee_to_hw_nozzle_geom0: origin xyz=0.029920000000000002 0.0 0.03517396538237974 rpy=0 -0.49514949 0 -> xyz=0.079 0.0 0.21311701994296112 rpy=0 -0.3154949 0
- joint ur_4_ee_to_hw_nozzle_geom1: origin xyz=0.021156634893101506 0.021156634893101503 0.03517396538237974 rpy=0 -0.49514949 0.7853981633974483 -> xyz=0.05586143571373726 0.05586143571373725 0.21311701994296112 rpy=0 -0.3154949 0.7853981633974483
- joint ur_4_ee_to_hw_nozzle_geom2: origin xyz=1.8320716115244406e-18 0.029920000000000002 0.03517396538237974 rpy=0 -0.49514949 1.5707963267948966 -> xyz=4.837354856632045e-18 0.079 0.21311701994296112 rpy=0 -0.3154949 1.5707963267948966
- joint ur_4_ee_to_hw_nozzle_geom3: origin xyz=-0.021156634893101503 0.021156634893101506 0.03517396538237974 rpy=0 -0.49514949 2.356194490192345 -> xyz=-0.05586143571373725 0.05586143571373726 0.21311701994296112 rpy=0 -0.3154949 2.356194490192345
- joint ur_4_ee_to_hw_nozzle_geom4: origin xyz=-0.029920000000000002 3.664143223048881e-18 0.03517396538237974 rpy=0 -0.49514949 3.141592653589793 -> xyz=-0.079 9.67470971326409e-18 0.21311701994296112 rpy=0 -0.3154949 3.141592653589793
- joint ur_4_ee_to_hw_nozzle_geom5: origin xyz=-0.021156634893101506 -0.021156634893101503 0.03517396538237974 rpy=0 -0.49514949 3.9269908169872414 -> xyz=-0.055861435713737265 -0.05586143571373725 0.21311701994296112 rpy=0 -0.3154949 3.9269908169872414
- joint ur_4_ee_to_hw_nozzle_geom6: origin xyz=-5.496214834573321e-18 -0.029920000000000002 0.03517396538237974 rpy=0 -0.49514949 4.71238898038469 -> xyz=-1.4512064569896134e-17 -0.079 0.21311701994296112 rpy=0 -0.3154949 4.71238898038469
- joint ur_4_ee_to_hw_nozzle_geom7: origin xyz=0.0211566348931015 -0.021156634893101506 0.03517396538237974 rpy=0 -0.49514949 5.497787143782138 -> xyz=0.055861435713737244 -0.055861435713737265 0.21311701994296112 rpy=0 -0.3154949 5.497787143782138
- joint ur_4_ee_to_tube_geom0: origin xyz=0.0127 0.0 0.08975 rpy=0 0 0 -> xyz=0.0127 0.0 0.45075 rpy=0 0 0
- joint ur_4_ee_to_tube_geom1: origin xyz=0.008980256121069154 0.008980256121069152 0.08975 rpy=0 0 0.7853981633974483 -> xyz=0.008980256121069154 0.008980256121069152 0.45075 rpy=0 0 0.7853981633974483
- joint ur_4_ee_to_tube_geom2: origin xyz=7.776507174585693e-19 0.0127 0.08975 rpy=0 0 1.5707963267948966 -> xyz=7.776507174585693e-19 0.0127 0.45075 rpy=0 0 1.5707963267948966
- joint ur_4_ee_to_tube_geom3: origin xyz=-0.008980256121069152 0.008980256121069154 0.08975 rpy=0 0 2.356194490192345 -> xyz=-0.008980256121069152 0.008980256121069154 0.45075 rpy=0 0 2.356194490192345
- joint ur_4_ee_to_tube_geom4: origin xyz=-0.0127 1.5553014349171385e-18 0.08975 rpy=0 0 3.141592653589793 -> xyz=-0.0127 1.5553014349171385e-18 0.45075 rpy=0 0 3.141592653589793
- joint ur_4_ee_to_tube_geom5: origin xyz=-0.008980256121069155 -0.008980256121069152 0.08975 rpy=0 0 3.9269908169872414 -> xyz=-0.008980256121069155 -0.008980256121069152 0.45075 rpy=0 0 3.9269908169872414
- joint ur_4_ee_to_tube_geom6: origin xyz=-2.3329521523757078e-18 -0.0127 0.08975 rpy=0 0 4.71238898038469 -> xyz=-2.3329521523757078e-18 -0.0127 0.45075 rpy=0 0 4.71238898038469
- joint ur_4_ee_to_tube_geom7: origin xyz=0.00898025612106915 -0.008980256121069155 0.08975 rpy=0 0 5.497787143782138 -> xyz=0.00898025612106915 -0.008980256121069155 0.45075 rpy=0 0 5.497787143782138
- joint ur_4_tool0_to_ee: origin xyz=0 0 0.12477 rpy=0 3.14159 0 -> xyz=0 0 0.4785 rpy=0 3.14159 0

File: urdf/simulation/satellite/cv.xacro (robot description, xacro)
@@ -10,7 +10,7 @@
   <link name="$(arg prefix)client">
     <visual>
-      <origin rpy="0 0 0" xyz="-0.048 -0.048 -1.9897"/>
+      <origin rpy="0 0 0" xyz="0 0 0"/>
       <geometry>
-        <mesh filename="package://on_orbit/urdf/simulation/meshes/cv_assembly.stl" scale="1 1 1"/>
+        <mesh filename="package://on_orbit/urdf/meshes/full_cv.stl" scale="1 1 1"/>
       </geometry>
       <material name="transparent_gray">
@@ -41,8 +41,8 @@
     <parent link="$(arg prefix)nozzle"/>
     <child link="$(arg prefix)capture_box"/>
-    <origin rpy="0 0 0" xyz="0 0 -0.451674428"/>
+    <origin rpy="0 0 0" xyz="0 0 -0.05"/>
   </joint>
   <link name="$(arg prefix)capture_box">
-  <!--<visual>
+  <!-- <visual>
       <origin rpy="0 0 0" xyz="0 0 0"/>
       <geometry>
@@ -52,5 +52,5 @@
         <color rgba="${rval} ${gval} ${bval} 0.0"/>
       </material>
-    </visual>-->
+    </visual> -->
     <inertial>
       <mass value="0"/>
@@ -71,5 +71,5 @@
     <parent link="$(arg prefix)nozzle"/>
     <child link="$(arg prefix)cone_vertex"/>
-    <origin rpy="0 0 0" xyz="0 0 0.0748"/>
+    <origin rpy="0 0 0" xyz="0 0 0"/>
   </joint>
   <link name="$(arg prefix)hole">
@@ -84,5 +84,5 @@
     <parent link="$(arg prefix)nozzle"/>
     <child link="$(arg prefix)hole"/>
-    <origin rpy="0 0 0" xyz="0 0 0.0675"/>
+    <origin rpy="0 0 0" xyz="0 0 0.429"/>
   </joint>
   <link name="$(arg prefix)goal">
@@ -97,5 +97,5 @@
     <parent link="$(arg prefix)nozzle"/>
     <child link="$(arg prefix)goal"/>
-    <origin rpy="0 0 0" xyz="0 0 0.110"/>
+    <origin rpy="0 0 0" xyz="0 0 0.4656"/>
   </joint>
   <link name="$(arg prefix)hole_end">
@@ -116,5 +116,5 @@
     <parent link="$(arg prefix)nozzle"/>
     <child link="$(arg prefix)hole_end"/>
-    <origin rpy="0 0 0" xyz="0 0 0.112"/>
+    <origin rpy="0 0 0" xyz="0 0 0.4785"/>
   </joint>
   <xacro:tube_geom num="0" theta="0" prefix="$(arg prefix)"/>

File: urdf/simulation/satellite/robot.xacro (robot description, xacro)
@@ -348,5 +348,5 @@
   <parent link="$(arg prefix)ee_body"/>
     <child link="$(arg prefix)ee_peg"/>
-    <origin rpy="0 0 0" xyz="0 0 1.1101"/>
+    <origin rpy="0 0 0" xyz="0 0 1.3101"/>
   </joint>
   <link name="$(arg prefix)ee_peg">

File: urdf/simulation/satellite/sim_nozzle_geom.xacro (robot description, xacro)
@@ -1,19 +1,18 @@
 <?xml version="1.0"?>
 <robot xmlns:xacro="http://www.ros.org/wiki/xacro">
-  <xacro:property name="nozzle_length" value="0.0675" />
-  <xacro:property name="nozzle_geom_length" value="0.07671" />
-  <xacro:property name="nozzle_wall_width" value="0.003" />
-  <xacro:property name="nozzle_box_width" value="0.04" />
-  <xacro:property name="throat_outer_diameter" value="0.028" />
+  <xacro:property name="nozzle_length" value="0.4285" />
+  <xacro:property name="nozzle_geom_length" value="0.4451" />
+  <xacro:property name="nozzle_wall_width" value="0.005" />
+  <xacro:property name="nozzle_box_width" value="0.125" />
+  <xacro:property name="throat_outer_diameter" value="0.032" />
   <xacro:property name="throat_middle_diameter" value="${throat_outer_diameter - nozzle_wall_width}" />
-  <xacro:property name="entry_outer_diameter" value="0.09768" />
+  <xacro:property name="entry_outer_diameter" value="0.294" />
   <xacro:property name="entry_middle_diameter" value="${entry_outer_diameter - nozzle_wall_width}" />
   <xacro:property name="entry_inner_rad" value="${(entry_outer_diameter - 2*nozzle_wall_width)/2}" />
   <xacro:property name="dist_from_centerline" value="${(throat_middle_diameter + entry_middle_diameter)/4}" />
-  <xacro:property name="slope_angle" value="0.49514949" />
+  <xacro:property name="slope_angle" value="0.3054949" />
   <xacro:macro name="nozzle_geom" params="num theta prefix">
     <link name="${prefix}nozzle_geom${num}">
-      <!--
-      <visual>
+      <!-- <visual>
         <origin rpy="0 0 0" xyz="0 0 0"/>
         <geometry>
@@ -23,6 +22,5 @@
           <color rgba="1.0 1.0 1.0 0.5"/>
         </material>
-      </visual>
-      -->
+      </visual> -->
       <inertial>
         <mass value="0"/>
