Commit message: urdf rebuilt

File: urdf/on_orbit_rail.urdf (robot description, URDF)
Before this commit: robot holodeck, 73 links, 72 joints
Links:
- removed link carriage_link_1
- removed link carriage_link_2
- removed link rail_1
- removed link ur_1_base
- removed link ur_1_base_link
- removed link ur_1_base_link_inertia
- removed link ur_1_flange
- removed link ur_1_forearm_link
- removed link ur_1_shoulder_link
- removed link ur_1_tool0
- removed link ur_1_upper_arm_link
- removed link ur_1_wrist_1_link
- removed link ur_1_wrist_2_link
- removed link ur_1_wrist_3_link
- removed link ur_2_base
- removed link ur_2_base_link
- removed link ur_2_base_link_inertia
- removed link ur_2_flange
- removed link ur_2_forearm_link
- removed link ur_2_shoulder_link
- removed link ur_2_tool0
- removed link ur_2_upper_arm_link
- removed link ur_2_wrist_1_link
- removed link ur_2_wrist_2_link
- removed link ur_2_wrist_3_link
Joints:
- removed joint carriage_1
- removed joint carriage_2
- removed joint fixed_1
- removed joint fixed_2
- removed joint fixed_rail_1
- removed joint ur_1_base_link-base_fixed_joint
- removed joint ur_1_base_link-base_link_inertia
- removed joint ur_1_elbow_joint
- removed joint ur_1_flange-tool0
- removed joint ur_1_shoulder_lift_joint
- removed joint ur_1_shoulder_pan_joint
- removed joint ur_1_wrist_1_joint
- removed joint ur_1_wrist_2_joint
- removed joint ur_1_wrist_3-flange
- removed joint ur_1_wrist_3_joint
- removed joint ur_2_base_link-base_fixed_joint
- removed joint ur_2_base_link-base_link_inertia
- removed joint ur_2_elbow_joint
- removed joint ur_2_flange-tool0
- removed joint ur_2_shoulder_lift_joint
- removed joint ur_2_shoulder_pan_joint
- removed joint ur_2_wrist_1_joint
- removed joint ur_2_wrist_2_joint
- removed joint ur_2_wrist_3-flange
- removed joint ur_2_wrist_3_joint
