Commit message: all urdf updated

File: urdf/holodeck.urdf (robot description, URDF)
Before this commit: robot holodeck, 73 links, 72 joints
Links:
- link ur_3_ee: mass 0.14597807959 -> 0.035; geometry collision cylinder length=0.1558 radius=0.0079; visual cylinder length=0.1558 radius=0.0079
Joints:
- joint ur_3_ee_to_peg_center: origin xyz=0 0 -0.1045 rpy=0 0 0 -> xyz=0 0 -0.0779 rpy=0 0 0
- joint ur_3_tool0_to_ee: origin xyz=0 0 0.209 rpy=0 0 0 -> xyz=0 0 0.1558 rpy=0 0 0
- joint ur_3_tool0_to_ft_sensor: origin xyz=0 0 0.0315 rpy=0 0 -0.53996123733 -> xyz=0 0 0.029 rpy=0 0 -0.53996123733
- joint ur_4_ee_to_goal: origin xyz=0 0 0.09017557238 rpy=0 3.141592653589793 0 -> xyz=0 0 0.11 rpy=0 3.141592653589793 0
- joint ur_4_tool0_to_ee: origin xyz=0 0 0.12477 rpy=0 3.14159 0 -> xyz=0 0 0.1194 rpy=0 3.14159 0

File: urdf/on_orbit_rail.urdf (robot description, URDF)
Before this commit: robot holodeck, 48 links, 47 joints
Links:
- link ur_3_ee: mass 0.14597807959 -> 0.035; geometry collision cylinder length=0.1558 radius=0.0079; visual cylinder length=0.1558 radius=0.0079
Joints:
- joint ur_3_ee_to_peg_center: origin xyz=0 0 -0.1045 rpy=0 0 0 -> xyz=0 0 -0.0779 rpy=0 0 0
- joint ur_3_tool0_to_ee: origin xyz=0 0 0.209 rpy=0 0 0 -> xyz=0 0 0.1558 rpy=0 0 0
- joint ur_3_tool0_to_ft_sensor: origin xyz=0 0 0.0315 rpy=0 0 -0.53996123733 -> xyz=0 0 0.029 rpy=0 0 -0.53996123733
- joint ur_4_ee_to_goal: origin xyz=0 0 0.09017557238 rpy=0 3.141592653589793 0 -> xyz=0 0 0.11 rpy=0 3.141592653589793 0
- joint ur_4_tool0_to_ee: origin xyz=0 0 0.12477 rpy=0 3.14159 0 -> xyz=0 0 0.1194 rpy=0 3.14159 0
