Commit message: couple changes before demo

File: urdf/cv.urdf (robot description, URDF)
Before this commit: robot FREND, 31 links, 30 joints
Links:
- link client: geometry visual mesh filename=package://on_orbit/urdf/meshes/full_cv.stl scale=1 1 1
- link nozzle_geom0: geometry collision box size=0.005 0.125 0.4451
- link nozzle_geom1: geometry collision box size=0.005 0.125 0.4451
- link nozzle_geom2: geometry collision box size=0.005 0.125 0.4451
- link nozzle_geom3: geometry collision box size=0.005 0.125 0.4451
- link nozzle_geom4: geometry collision box size=0.005 0.125 0.4451
- link nozzle_geom5: geometry collision box size=0.005 0.125 0.4451
- link nozzle_geom6: geometry collision box size=0.005 0.125 0.4451
- link nozzle_geom7: geometry collision box size=0.005 0.125 0.4451
Joints:
- joint nozzle_to_capture_box: origin xyz=0 0 -0.451674428 rpy=0 0 0 -> xyz=0 0 -0.05 rpy=0 0 0
- joint nozzle_to_cone_vertex: origin xyz=0 0 0.0748 rpy=0 0 0 -> xyz=0 0 0 rpy=0 0 0
- joint nozzle_to_goal: origin xyz=0 0 0.110 rpy=0 0 0 -> xyz=0 0 0.4656 rpy=0 0 0
- joint nozzle_to_hole: origin xyz=0 0 0.0675 rpy=0 0 0 -> xyz=0 0 0.429 rpy=0 0 0
- joint nozzle_to_hole_end: origin xyz=0 0 0.112 rpy=0 0 0 -> xyz=0 0 0.4785 rpy=0 0 0
- joint nozzle_to_nozzle_geom0: origin xyz=0.029920000000000002 0.0 0.03517396538237974 rpy=0 -0.49514949 0 -> xyz=0.079 0.0 0.21374936499656222 rpy=0 -0.3054949 0
- joint nozzle_to_nozzle_geom1: origin xyz=0.021156634893101506 0.021156634893101503 0.03517396538237974 rpy=0 -0.49514949 0.7853981633974483 -> xyz=0.05586143571373726 0.05586143571373725 0.21374936499656222 rpy=0 -0.3054949 0.7853981633974483
- joint nozzle_to_nozzle_geom2: origin xyz=1.8320716115244406e-18 0.029920000000000002 0.03517396538237974 rpy=0 -0.49514949 1.5707963267948966 -> xyz=4.837354856632045e-18 0.079 0.21374936499656222 rpy=0 -0.3054949 1.5707963267948966
- joint nozzle_to_nozzle_geom3: origin xyz=-0.021156634893101503 0.021156634893101506 0.03517396538237974 rpy=0 -0.49514949 2.356194490192345 -> xyz=-0.05586143571373725 0.05586143571373726 0.21374936499656222 rpy=0 -0.3054949 2.356194490192345
- joint nozzle_to_nozzle_geom4: origin xyz=-0.029920000000000002 3.664143223048881e-18 0.03517396538237974 rpy=0 -0.49514949 3.141592653589793 -> xyz=-0.079 9.67470971326409e-18 0.21374936499656222 rpy=0 -0.3054949 3.141592653589793
- joint nozzle_to_nozzle_geom5: origin xyz=-0.021156634893101506 -0.021156634893101503 0.03517396538237974 rpy=0 -0.49514949 3.9269908169872414 -> xyz=-0.055861435713737265 -0.05586143571373725 0.21374936499656222 rpy=0 -0.3054949 3.9269908169872414
- joint nozzle_to_nozzle_geom6: origin xyz=-5.496214834573321e-18 -0.029920000000000002 0.03517396538237974 rpy=0 -0.49514949 4.71238898038469 -> xyz=-1.4512064569896134e-17 -0.079 0.21374936499656222 rpy=0 -0.3054949 4.71238898038469
- joint nozzle_to_nozzle_geom7: origin xyz=0.0211566348931015 -0.021156634893101506 0.03517396538237974 rpy=0 -0.49514949 5.497787143782138 -> xyz=0.055861435713737244 -0.055861435713737265 0.21374936499656222 rpy=0 -0.3054949 5.497787143782138
- joint nozzle_to_nozzle_rim0: origin xyz=0.04584 0.0 0 rpy=0 -0.49514949 0 -> xyz=0.142 0.0 0 rpy=0 -0.3054949 0
- joint nozzle_to_nozzle_rim1: origin xyz=0.03241377484959134 0.032413774849591334 0 rpy=0 -0.49514949 0.7853981633974483 -> xyz=0.10040916292848974 0.10040916292848973 0 rpy=0 -0.3054949 0.7853981633974483
- joint nozzle_to_nozzle_rim2: origin xyz=2.8068904636457335e-18 0.04584 0 rpy=0 -0.49514949 1.5707963267948966 -> xyz=8.694992273946207e-18 0.142 0 rpy=0 -0.3054949 1.5707963267948966
- joint nozzle_to_nozzle_rim3: origin xyz=-0.032413774849591334 0.03241377484959134 0 rpy=0 -0.49514949 2.356194490192345 -> xyz=-0.10040916292848973 0.10040916292848974 0 rpy=0 -0.3054949 2.356194490192345
- joint nozzle_to_nozzle_rim4: origin xyz=-0.04584 5.613780927291467e-18 0 rpy=0 -0.49514949 3.141592653589793 -> xyz=-0.142 1.7389984547892414e-17 0 rpy=0 -0.3054949 3.141592653589793
- joint nozzle_to_nozzle_rim5: origin xyz=-0.03241377484959135 -0.032413774849591334 0 rpy=0 -0.49514949 3.9269908169872414 -> xyz=-0.10040916292848977 -0.10040916292848973 0 rpy=0 -0.3054949 3.9269908169872414
- joint nozzle_to_nozzle_rim6: origin xyz=-8.4206713909372e-18 -0.04584 0 rpy=0 -0.49514949 4.71238898038469 -> xyz=-2.6084976821838618e-17 -0.142 0 rpy=0 -0.3054949 4.71238898038469
- joint nozzle_to_nozzle_rim7: origin xyz=0.03241377484959133 -0.03241377484959135 0 rpy=0 -0.49514949 5.497787143782138 -> xyz=0.10040916292848971 -0.10040916292848977 0 rpy=0 -0.3054949 5.497787143782138
- joint nozzle_to_tube_geom0: origin xyz=0.0127 0.0 0.08975 rpy=0 0 0 -> xyz=0.0127 0.0 0.45075 rpy=0 0 0
- joint nozzle_to_tube_geom1: origin xyz=0.008980256121069154 0.008980256121069152 0.08975 rpy=0 0 0.7853981633974483 -> xyz=0.008980256121069154 0.008980256121069152 0.45075 rpy=0 0 0.7853981633974483
- joint nozzle_to_tube_geom2: origin xyz=7.776507174585693e-19 0.0127 0.08975 rpy=0 0 1.5707963267948966 -> xyz=7.776507174585693e-19 0.0127 0.45075 rpy=0 0 1.5707963267948966
- joint nozzle_to_tube_geom3: origin xyz=-0.008980256121069152 0.008980256121069154 0.08975 rpy=0 0 2.356194490192345 -> xyz=-0.008980256121069152 0.008980256121069154 0.45075 rpy=0 0 2.356194490192345
- joint nozzle_to_tube_geom4: origin xyz=-0.0127 1.5553014349171385e-18 0.08975 rpy=0 0 3.141592653589793 -> xyz=-0.0127 1.5553014349171385e-18 0.45075 rpy=0 0 3.141592653589793
- joint nozzle_to_tube_geom5: origin xyz=-0.008980256121069155 -0.008980256121069152 0.08975 rpy=0 0 3.9269908169872414 -> xyz=-0.008980256121069155 -0.008980256121069152 0.45075 rpy=0 0 3.9269908169872414
- joint nozzle_to_tube_geom6: origin xyz=-2.3329521523757078e-18 -0.0127 0.08975 rpy=0 0 4.71238898038469 -> xyz=-2.3329521523757078e-18 -0.0127 0.45075 rpy=0 0 4.71238898038469
- joint nozzle_to_tube_geom7: origin xyz=0.00898025612106915 -0.008980256121069155 0.08975 rpy=0 0 5.497787143782138 -> xyz=0.00898025612106915 -0.008980256121069155 0.45075 rpy=0 0 5.497787143782138

File: urdf/robot_cv_detached.urdf (robot description, URDF)
Before this commit: robot FREND, 48 links, 47 joints
Links:
- link client: geometry visual mesh filename=package://on_orbit/urdf/meshes/full_cv.stl scale=1 1 1
- link nozzle_geom0: geometry collision box size=0.005 0.125 0.4451
- link nozzle_geom1: geometry collision box size=0.005 0.125 0.4451
- link nozzle_geom2: geometry collision box size=0.005 0.125 0.4451
- link nozzle_geom3: geometry collision box size=0.005 0.125 0.4451
- link nozzle_geom4: geometry collision box size=0.005 0.125 0.4451
- link nozzle_geom5: geometry collision box size=0.005 0.125 0.4451
- link nozzle_geom6: geometry collision box size=0.005 0.125 0.4451
- link nozzle_geom7: geometry collision box size=0.005 0.125 0.4451
Joints:
- joint ee_peg_joint: origin xyz=0 0 1.1101 rpy=0 0 0 -> xyz=0 0 1.3101 rpy=0 0 0
- joint nozzle_to_capture_box: origin xyz=0 0 -0.451674428 rpy=0 0 0 -> xyz=0 0 -0.05 rpy=0 0 0
- joint nozzle_to_cone_vertex: origin xyz=0 0 0.0748 rpy=0 0 0 -> xyz=0 0 0 rpy=0 0 0
- joint nozzle_to_goal: origin xyz=0 0 0.110 rpy=0 0 0 -> xyz=0 0 0.4656 rpy=0 0 0
- joint nozzle_to_hole: origin xyz=0 0 0.0675 rpy=0 0 0 -> xyz=0 0 0.429 rpy=0 0 0
- joint nozzle_to_hole_end: origin xyz=0 0 0.112 rpy=0 0 0 -> xyz=0 0 0.4785 rpy=0 0 0
- joint nozzle_to_nozzle_geom0: origin xyz=0.029920000000000002 0.0 0.03517396538237974 rpy=0 -0.49514949 0 -> xyz=0.079 0.0 0.21374936499656222 rpy=0 -0.3054949 0
- joint nozzle_to_nozzle_geom1: origin xyz=0.021156634893101506 0.021156634893101503 0.03517396538237974 rpy=0 -0.49514949 0.7853981633974483 -> xyz=0.05586143571373726 0.05586143571373725 0.21374936499656222 rpy=0 -0.3054949 0.7853981633974483
- joint nozzle_to_nozzle_geom2: origin xyz=1.8320716115244406e-18 0.029920000000000002 0.03517396538237974 rpy=0 -0.49514949 1.5707963267948966 -> xyz=4.837354856632045e-18 0.079 0.21374936499656222 rpy=0 -0.3054949 1.5707963267948966
- joint nozzle_to_nozzle_geom3: origin xyz=-0.021156634893101503 0.021156634893101506 0.03517396538237974 rpy=0 -0.49514949 2.356194490192345 -> xyz=-0.05586143571373725 0.05586143571373726 0.21374936499656222 rpy=0 -0.3054949 2.356194490192345
- joint nozzle_to_nozzle_geom4: origin xyz=-0.029920000000000002 3.664143223048881e-18 0.03517396538237974 rpy=0 -0.49514949 3.141592653589793 -> xyz=-0.079 9.67470971326409e-18 0.21374936499656222 rpy=0 -0.3054949 3.141592653589793
- joint nozzle_to_nozzle_geom5: origin xyz=-0.021156634893101506 -0.021156634893101503 0.03517396538237974 rpy=0 -0.49514949 3.9269908169872414 -> xyz=-0.055861435713737265 -0.05586143571373725 0.21374936499656222 rpy=0 -0.3054949 3.9269908169872414
- joint nozzle_to_nozzle_geom6: origin xyz=-5.496214834573321e-18 -0.029920000000000002 0.03517396538237974 rpy=0 -0.49514949 4.71238898038469 -> xyz=-1.4512064569896134e-17 -0.079 0.21374936499656222 rpy=0 -0.3054949 4.71238898038469
- joint nozzle_to_nozzle_geom7: origin xyz=0.0211566348931015 -0.021156634893101506 0.03517396538237974 rpy=0 -0.49514949 5.497787143782138 -> xyz=0.055861435713737244 -0.055861435713737265 0.21374936499656222 rpy=0 -0.3054949 5.497787143782138
- joint nozzle_to_nozzle_rim0: origin xyz=0.04584 0.0 0 rpy=0 -0.49514949 0 -> xyz=0.142 0.0 0 rpy=0 -0.3054949 0
- joint nozzle_to_nozzle_rim1: origin xyz=0.03241377484959134 0.032413774849591334 0 rpy=0 -0.49514949 0.7853981633974483 -> xyz=0.10040916292848974 0.10040916292848973 0 rpy=0 -0.3054949 0.7853981633974483
- joint nozzle_to_nozzle_rim2: origin xyz=2.8068904636457335e-18 0.04584 0 rpy=0 -0.49514949 1.5707963267948966 -> xyz=8.694992273946207e-18 0.142 0 rpy=0 -0.3054949 1.5707963267948966
- joint nozzle_to_nozzle_rim3: origin xyz=-0.032413774849591334 0.03241377484959134 0 rpy=0 -0.49514949 2.356194490192345 -> xyz=-0.10040916292848973 0.10040916292848974 0 rpy=0 -0.3054949 2.356194490192345
- joint nozzle_to_nozzle_rim4: origin xyz=-0.04584 5.613780927291467e-18 0 rpy=0 -0.49514949 3.141592653589793 -> xyz=-0.142 1.7389984547892414e-17 0 rpy=0 -0.3054949 3.141592653589793
- joint nozzle_to_nozzle_rim5: origin xyz=-0.03241377484959135 -0.032413774849591334 0 rpy=0 -0.49514949 3.9269908169872414 -> xyz=-0.10040916292848977 -0.10040916292848973 0 rpy=0 -0.3054949 3.9269908169872414
- joint nozzle_to_nozzle_rim6: origin xyz=-8.4206713909372e-18 -0.04584 0 rpy=0 -0.49514949 4.71238898038469 -> xyz=-2.6084976821838618e-17 -0.142 0 rpy=0 -0.3054949 4.71238898038469
- joint nozzle_to_nozzle_rim7: origin xyz=0.03241377484959133 -0.03241377484959135 0 rpy=0 -0.49514949 5.497787143782138 -> xyz=0.10040916292848971 -0.10040916292848977 0 rpy=0 -0.3054949 5.497787143782138
- joint nozzle_to_tube_geom0: origin xyz=0.0127 0.0 0.08975 rpy=0 0 0 -> xyz=0.0127 0.0 0.45075 rpy=0 0 0
- joint nozzle_to_tube_geom1: origin xyz=0.008980256121069154 0.008980256121069152 0.08975 rpy=0 0 0.7853981633974483 -> xyz=0.008980256121069154 0.008980256121069152 0.45075 rpy=0 0 0.7853981633974483
- joint nozzle_to_tube_geom2: origin xyz=7.776507174585693e-19 0.0127 0.08975 rpy=0 0 1.5707963267948966 -> xyz=7.776507174585693e-19 0.0127 0.45075 rpy=0 0 1.5707963267948966
- joint nozzle_to_tube_geom3: origin xyz=-0.008980256121069152 0.008980256121069154 0.08975 rpy=0 0 2.356194490192345 -> xyz=-0.008980256121069152 0.008980256121069154 0.45075 rpy=0 0 2.356194490192345
- joint nozzle_to_tube_geom4: origin xyz=-0.0127 1.5553014349171385e-18 0.08975 rpy=0 0 3.141592653589793 -> xyz=-0.0127 1.5553014349171385e-18 0.45075 rpy=0 0 3.141592653589793
- joint nozzle_to_tube_geom5: origin xyz=-0.008980256121069155 -0.008980256121069152 0.08975 rpy=0 0 3.9269908169872414 -> xyz=-0.008980256121069155 -0.008980256121069152 0.45075 rpy=0 0 3.9269908169872414
- joint nozzle_to_tube_geom6: origin xyz=-2.3329521523757078e-18 -0.0127 0.08975 rpy=0 0 4.71238898038469 -> xyz=-2.3329521523757078e-18 -0.0127 0.45075 rpy=0 0 4.71238898038469
- joint nozzle_to_tube_geom7: origin xyz=0.00898025612106915 -0.008980256121069155 0.08975 rpy=0 0 5.497787143782138 -> xyz=0.00898025612106915 -0.008980256121069155 0.45075 rpy=0 0 5.497787143782138
