Commit message: updated visualization things to make on_orbit viz display live state

File: urdf/cv.urdf (robot description, URDF)
Before this commit: robot FREND, 31 links, 30 joints
Links:
- link nozzle_geom0: geometry collision box size=0.005 0.125 0.4551
- link nozzle_geom1: geometry collision box size=0.005 0.125 0.4551
- link nozzle_geom2: geometry collision box size=0.005 0.125 0.4551
- link nozzle_geom3: geometry collision box size=0.005 0.125 0.4551
- link nozzle_geom4: geometry collision box size=0.005 0.125 0.4551
- link nozzle_geom5: geometry collision box size=0.005 0.125 0.4551
- link nozzle_geom6: geometry collision box size=0.005 0.125 0.4551
- link nozzle_geom7: geometry collision box size=0.005 0.125 0.4551
Joints:
- joint nozzle_to_nozzle_geom0: origin xyz=0.079 0.0 0.21374936499656222 rpy=0 -0.3054949 0 -> xyz=0.079 0.0 0.2184025683012885 rpy=0 -0.3073 0
- joint nozzle_to_nozzle_geom1: origin xyz=0.05586143571373726 0.05586143571373725 0.21374936499656222 rpy=0 -0.3054949 0.7853981633974483 -> xyz=0.05586143571373726 0.05586143571373725 0.2184025683012885 rpy=0 -0.3073 0.7853981633974483
- joint nozzle_to_nozzle_geom2: origin xyz=4.837354856632045e-18 0.079 0.21374936499656222 rpy=0 -0.3054949 1.5707963267948966 -> xyz=4.837354856632045e-18 0.079 0.2184025683012885 rpy=0 -0.3073 1.5707963267948966
- joint nozzle_to_nozzle_geom3: origin xyz=-0.05586143571373725 0.05586143571373726 0.21374936499656222 rpy=0 -0.3054949 2.356194490192345 -> xyz=-0.05586143571373725 0.05586143571373726 0.2184025683012885 rpy=0 -0.3073 2.356194490192345
- joint nozzle_to_nozzle_geom4: origin xyz=-0.079 9.67470971326409e-18 0.21374936499656222 rpy=0 -0.3054949 3.141592653589793 -> xyz=-0.079 9.67470971326409e-18 0.2184025683012885 rpy=0 -0.3073 3.141592653589793
- joint nozzle_to_nozzle_geom5: origin xyz=-0.055861435713737265 -0.05586143571373725 0.21374936499656222 rpy=0 -0.3054949 3.9269908169872414 -> xyz=-0.055861435713737265 -0.05586143571373725 0.2184025683012885 rpy=0 -0.3073 3.9269908169872414
- joint nozzle_to_nozzle_geom6: origin xyz=-1.4512064569896134e-17 -0.079 0.21374936499656222 rpy=0 -0.3054949 4.71238898038469 -> xyz=-1.4512064569896134e-17 -0.079 0.2184025683012885 rpy=0 -0.3073 4.71238898038469
- joint nozzle_to_nozzle_geom7: origin xyz=0.055861435713737244 -0.055861435713737265 0.21374936499656222 rpy=0 -0.3054949 5.497787143782138 -> xyz=0.055861435713737244 -0.055861435713737265 0.2184025683012885 rpy=0 -0.3073 5.497787143782138
- joint nozzle_to_nozzle_rim0: origin xyz=0.142 0.0 0 rpy=0 -0.3054949 0 -> xyz=0.142 0.0 0 rpy=0 -0.3073 0
- joint nozzle_to_nozzle_rim1: origin xyz=0.10040916292848974 0.10040916292848973 0 rpy=0 -0.3054949 0.7853981633974483 -> xyz=0.10040916292848974 0.10040916292848973 0 rpy=0 -0.3073 0.7853981633974483
- joint nozzle_to_nozzle_rim2: origin xyz=8.694992273946207e-18 0.142 0 rpy=0 -0.3054949 1.5707963267948966 -> xyz=8.694992273946207e-18 0.142 0 rpy=0 -0.3073 1.5707963267948966
- joint nozzle_to_nozzle_rim3: origin xyz=-0.10040916292848973 0.10040916292848974 0 rpy=0 -0.3054949 2.356194490192345 -> xyz=-0.10040916292848973 0.10040916292848974 0 rpy=0 -0.3073 2.356194490192345
- joint nozzle_to_nozzle_rim4: origin xyz=-0.142 1.7389984547892414e-17 0 rpy=0 -0.3054949 3.141592653589793 -> xyz=-0.142 1.7389984547892414e-17 0 rpy=0 -0.3073 3.141592653589793
- joint nozzle_to_nozzle_rim5: origin xyz=-0.10040916292848977 -0.10040916292848973 0 rpy=0 -0.3054949 3.9269908169872414 -> xyz=-0.10040916292848977 -0.10040916292848973 0 rpy=0 -0.3073 3.9269908169872414
- joint nozzle_to_nozzle_rim6: origin xyz=-2.6084976821838618e-17 -0.142 0 rpy=0 -0.3054949 4.71238898038469 -> xyz=-2.6084976821838618e-17 -0.142 0 rpy=0 -0.3073 4.71238898038469
- joint nozzle_to_nozzle_rim7: origin xyz=0.10040916292848971 -0.10040916292848977 0 rpy=0 -0.3054949 5.497787143782138 -> xyz=0.10040916292848971 -0.10040916292848977 0 rpy=0 -0.3073 5.497787143782138

File: urdf/hardware/ur/hw_nozzle_geom.xacro (robot description, xacro)
@@ -2,5 +2,5 @@
 <robot xmlns:xacro="http://www.ros.org/wiki/xacro">
   <xacro:property name="nozzle_length" value="0.4285" />
-  <xacro:property name="nozzle_geom_length" value="0.4451" />
+  <xacro:property name="nozzle_geom_length" value="0.4551" />
   <xacro:property name="nozzle_wall_width" value="0.005" />
   <xacro:property name="nozzle_box_width" value="0.125" />
@@ -11,5 +11,5 @@
   <xacro:property name="entry_inner_rad" value="${(entry_outer_diameter - 2*nozzle_wall_width)/2}" />
   <xacro:property name="dist_from_centerline" value="${(throat_middle_diameter + entry_middle_diameter)/4}" />
-  <xacro:property name="slope_angle" value="0.3154949" />
+  <xacro:property name="slope_angle" value="0.3073" />
   <xacro:macro name="hw_nozzle_geom" params="num theta">
     <link name="hw_nozzle_geom${num}">

File: urdf/holodeck.urdf (robot description, URDF)
Before this commit: robot holodeck, 73 links, 72 joints
Links:
- link hw_nozzle_geom0: geometry collision box size=0.005 0.125 0.4551; visual box size=0.005 0.125 0.4551
- link hw_nozzle_geom1: geometry collision box size=0.005 0.125 0.4551; visual box size=0.005 0.125 0.4551
- link hw_nozzle_geom2: geometry collision box size=0.005 0.125 0.4551; visual box size=0.005 0.125 0.4551
- link hw_nozzle_geom3: geometry collision box size=0.005 0.125 0.4551; visual box size=0.005 0.125 0.4551
- link hw_nozzle_geom4: geometry collision box size=0.005 0.125 0.4551; visual box size=0.005 0.125 0.4551
- link hw_nozzle_geom5: geometry collision box size=0.005 0.125 0.4551; visual box size=0.005 0.125 0.4551
- link hw_nozzle_geom6: geometry collision box size=0.005 0.125 0.4551; visual box size=0.005 0.125 0.4551
- link hw_nozzle_geom7: geometry collision box size=0.005 0.125 0.4551; visual box size=0.005 0.125 0.4551
Joints:
- joint ur_4_ee_to_hw_nozzle_geom0: origin xyz=0.079 0.0 0.21311701994296112 rpy=0 -0.3154949 0 -> xyz=0.079 0.0 0.2184025683012885 rpy=0 -0.3073 0
- joint ur_4_ee_to_hw_nozzle_geom1: origin xyz=0.05586143571373726 0.05586143571373725 0.21311701994296112 rpy=0 -0.3154949 0.7853981633974483 -> xyz=0.05586143571373726 0.05586143571373725 0.2184025683012885 rpy=0 -0.3073 0.7853981633974483
- joint ur_4_ee_to_hw_nozzle_geom2: origin xyz=4.837354856632045e-18 0.079 0.21311701994296112 rpy=0 -0.3154949 1.5707963267948966 -> xyz=4.837354856632045e-18 0.079 0.2184025683012885 rpy=0 -0.3073 1.5707963267948966
- joint ur_4_ee_to_hw_nozzle_geom3: origin xyz=-0.05586143571373725 0.05586143571373726 0.21311701994296112 rpy=0 -0.3154949 2.356194490192345 -> xyz=-0.05586143571373725 0.05586143571373726 0.2184025683012885 rpy=0 -0.3073 2.356194490192345
- joint ur_4_ee_to_hw_nozzle_geom4: origin xyz=-0.079 9.67470971326409e-18 0.21311701994296112 rpy=0 -0.3154949 3.141592653589793 -> xyz=-0.079 9.67470971326409e-18 0.2184025683012885 rpy=0 -0.3073 3.141592653589793
- joint ur_4_ee_to_hw_nozzle_geom5: origin xyz=-0.055861435713737265 -0.05586143571373725 0.21311701994296112 rpy=0 -0.3154949 3.9269908169872414 -> xyz=-0.055861435713737265 -0.05586143571373725 0.2184025683012885 rpy=0 -0.3073 3.9269908169872414
- joint ur_4_ee_to_hw_nozzle_geom6: origin xyz=-1.4512064569896134e-17 -0.079 0.21311701994296112 rpy=0 -0.3154949 4.71238898038469 -> xyz=-1.4512064569896134e-17 -0.079 0.2184025683012885 rpy=0 -0.3073 4.71238898038469
- joint ur_4_ee_to_hw_nozzle_geom7: origin xyz=0.055861435713737244 -0.055861435713737265 0.21311701994296112 rpy=0 -0.3154949 5.497787143782138 -> xyz=0.055861435713737244 -0.055861435713737265 0.2184025683012885 rpy=0 -0.3073 5.497787143782138

File: urdf/on_orbit.urdf (robot description, URDF)
Before this commit: robot holodeck, 48 links, 47 joints
Links:
- link hw_nozzle_geom0: geometry collision box size=0.005 0.125 0.4551; visual box size=0.005 0.125 0.4551
- link hw_nozzle_geom1: geometry collision box size=0.005 0.125 0.4551; visual box size=0.005 0.125 0.4551
- link hw_nozzle_geom2: geometry collision box size=0.005 0.125 0.4551; visual box size=0.005 0.125 0.4551
- link hw_nozzle_geom3: geometry collision box size=0.005 0.125 0.4551; visual box size=0.005 0.125 0.4551
- link hw_nozzle_geom4: geometry collision box size=0.005 0.125 0.4551; visual box size=0.005 0.125 0.4551
- link hw_nozzle_geom5: geometry collision box size=0.005 0.125 0.4551; visual box size=0.005 0.125 0.4551
- link hw_nozzle_geom6: geometry collision box size=0.005 0.125 0.4551; visual box size=0.005 0.125 0.4551
- link hw_nozzle_geom7: geometry collision box size=0.005 0.125 0.4551; visual box size=0.005 0.125 0.4551
Joints:
- joint ur_4_ee_to_hw_nozzle_geom0: origin xyz=0.079 0.0 0.21311701994296112 rpy=0 -0.3154949 0 -> xyz=0.079 0.0 0.2184025683012885 rpy=0 -0.3073 0
- joint ur_4_ee_to_hw_nozzle_geom1: origin xyz=0.05586143571373726 0.05586143571373725 0.21311701994296112 rpy=0 -0.3154949 0.7853981633974483 -> xyz=0.05586143571373726 0.05586143571373725 0.2184025683012885 rpy=0 -0.3073 0.7853981633974483
- joint ur_4_ee_to_hw_nozzle_geom2: origin xyz=4.837354856632045e-18 0.079 0.21311701994296112 rpy=0 -0.3154949 1.5707963267948966 -> xyz=4.837354856632045e-18 0.079 0.2184025683012885 rpy=0 -0.3073 1.5707963267948966
- joint ur_4_ee_to_hw_nozzle_geom3: origin xyz=-0.05586143571373725 0.05586143571373726 0.21311701994296112 rpy=0 -0.3154949 2.356194490192345 -> xyz=-0.05586143571373725 0.05586143571373726 0.2184025683012885 rpy=0 -0.3073 2.356194490192345
- joint ur_4_ee_to_hw_nozzle_geom4: origin xyz=-0.079 9.67470971326409e-18 0.21311701994296112 rpy=0 -0.3154949 3.141592653589793 -> xyz=-0.079 9.67470971326409e-18 0.2184025683012885 rpy=0 -0.3073 3.141592653589793
- joint ur_4_ee_to_hw_nozzle_geom5: origin xyz=-0.055861435713737265 -0.05586143571373725 0.21311701994296112 rpy=0 -0.3154949 3.9269908169872414 -> xyz=-0.055861435713737265 -0.05586143571373725 0.2184025683012885 rpy=0 -0.3073 3.9269908169872414
- joint ur_4_ee_to_hw_nozzle_geom6: origin xyz=-1.4512064569896134e-17 -0.079 0.21311701994296112 rpy=0 -0.3154949 4.71238898038469 -> xyz=-1.4512064569896134e-17 -0.079 0.2184025683012885 rpy=0 -0.3073 4.71238898038469
- joint ur_4_ee_to_hw_nozzle_geom7: origin xyz=0.055861435713737244 -0.055861435713737265 0.21311701994296112 rpy=0 -0.3154949 5.497787143782138 -> xyz=0.055861435713737244 -0.055861435713737265 0.2184025683012885 rpy=0 -0.3073 5.497787143782138

File: urdf/robot.urdf (robot description, URDF)
Before this commit: robot FREND, 16 links, 15 joints
Joints:
- joint ee_peg_joint: origin xyz=0 0 1.1101 rpy=0 0 0 -> xyz=0 0 1.3101 rpy=0 0 0

File: urdf/robot_cv_detached.urdf (robot description, URDF)
Before this commit: robot FREND, 48 links, 47 joints
Links:
- link nozzle_geom0: geometry collision box size=0.005 0.125 0.4551
- link nozzle_geom1: geometry collision box size=0.005 0.125 0.4551
- link nozzle_geom2: geometry collision box size=0.005 0.125 0.4551
- link nozzle_geom3: geometry collision box size=0.005 0.125 0.4551
- link nozzle_geom4: geometry collision box size=0.005 0.125 0.4551
- link nozzle_geom5: geometry collision box size=0.005 0.125 0.4551
- link nozzle_geom6: geometry collision box size=0.005 0.125 0.4551
- link nozzle_geom7: geometry collision box size=0.005 0.125 0.4551
Joints:
- joint nozzle_to_nozzle_geom0: origin xyz=0.079 0.0 0.21374936499656222 rpy=0 -0.3054949 0 -> xyz=0.079 0.0 0.2184025683012885 rpy=0 -0.3073 0
- joint nozzle_to_nozzle_geom1: origin xyz=0.05586143571373726 0.05586143571373725 0.21374936499656222 rpy=0 -0.3054949 0.7853981633974483 -> xyz=0.05586143571373726 0.05586143571373725 0.2184025683012885 rpy=0 -0.3073 0.7853981633974483
- joint nozzle_to_nozzle_geom2: origin xyz=4.837354856632045e-18 0.079 0.21374936499656222 rpy=0 -0.3054949 1.5707963267948966 -> xyz=4.837354856632045e-18 0.079 0.2184025683012885 rpy=0 -0.3073 1.5707963267948966
- joint nozzle_to_nozzle_geom3: origin xyz=-0.05586143571373725 0.05586143571373726 0.21374936499656222 rpy=0 -0.3054949 2.356194490192345 -> xyz=-0.05586143571373725 0.05586143571373726 0.2184025683012885 rpy=0 -0.3073 2.356194490192345
- joint nozzle_to_nozzle_geom4: origin xyz=-0.079 9.67470971326409e-18 0.21374936499656222 rpy=0 -0.3054949 3.141592653589793 -> xyz=-0.079 9.67470971326409e-18 0.2184025683012885 rpy=0 -0.3073 3.141592653589793
- joint nozzle_to_nozzle_geom5: origin xyz=-0.055861435713737265 -0.05586143571373725 0.21374936499656222 rpy=0 -0.3054949 3.9269908169872414 -> xyz=-0.055861435713737265 -0.05586143571373725 0.2184025683012885 rpy=0 -0.3073 3.9269908169872414
- joint nozzle_to_nozzle_geom6: origin xyz=-1.4512064569896134e-17 -0.079 0.21374936499656222 rpy=0 -0.3054949 4.71238898038469 -> xyz=-1.4512064569896134e-17 -0.079 0.2184025683012885 rpy=0 -0.3073 4.71238898038469
- joint nozzle_to_nozzle_geom7: origin xyz=0.055861435713737244 -0.055861435713737265 0.21374936499656222 rpy=0 -0.3054949 5.497787143782138 -> xyz=0.055861435713737244 -0.055861435713737265 0.2184025683012885 rpy=0 -0.3073 5.497787143782138
- joint nozzle_to_nozzle_rim0: origin xyz=0.142 0.0 0 rpy=0 -0.3054949 0 -> xyz=0.142 0.0 0 rpy=0 -0.3073 0
- joint nozzle_to_nozzle_rim1: origin xyz=0.10040916292848974 0.10040916292848973 0 rpy=0 -0.3054949 0.7853981633974483 -> xyz=0.10040916292848974 0.10040916292848973 0 rpy=0 -0.3073 0.7853981633974483
- joint nozzle_to_nozzle_rim2: origin xyz=8.694992273946207e-18 0.142 0 rpy=0 -0.3054949 1.5707963267948966 -> xyz=8.694992273946207e-18 0.142 0 rpy=0 -0.3073 1.5707963267948966
- joint nozzle_to_nozzle_rim3: origin xyz=-0.10040916292848973 0.10040916292848974 0 rpy=0 -0.3054949 2.356194490192345 -> xyz=-0.10040916292848973 0.10040916292848974 0 rpy=0 -0.3073 2.356194490192345
- joint nozzle_to_nozzle_rim4: origin xyz=-0.142 1.7389984547892414e-17 0 rpy=0 -0.3054949 3.141592653589793 -> xyz=-0.142 1.7389984547892414e-17 0 rpy=0 -0.3073 3.141592653589793
- joint nozzle_to_nozzle_rim5: origin xyz=-0.10040916292848977 -0.10040916292848973 0 rpy=0 -0.3054949 3.9269908169872414 -> xyz=-0.10040916292848977 -0.10040916292848973 0 rpy=0 -0.3073 3.9269908169872414
- joint nozzle_to_nozzle_rim6: origin xyz=-2.6084976821838618e-17 -0.142 0 rpy=0 -0.3054949 4.71238898038469 -> xyz=-2.6084976821838618e-17 -0.142 0 rpy=0 -0.3073 4.71238898038469
- joint nozzle_to_nozzle_rim7: origin xyz=0.10040916292848971 -0.10040916292848977 0 rpy=0 -0.3054949 5.497787143782138 -> xyz=0.10040916292848971 -0.10040916292848977 0 rpy=0 -0.3073 5.497787143782138

File: urdf/simulation/satellite/sim_nozzle_geom.xacro (robot description, xacro)
@@ -2,5 +2,5 @@
 <robot xmlns:xacro="http://www.ros.org/wiki/xacro">
   <xacro:property name="nozzle_length" value="0.4285" />
-  <xacro:property name="nozzle_geom_length" value="0.4451" />
+  <xacro:property name="nozzle_geom_length" value="0.4551" />
   <xacro:property name="nozzle_wall_width" value="0.005" />
   <xacro:property name="nozzle_box_width" value="0.125" />
@@ -11,5 +11,5 @@
   <xacro:property name="entry_inner_rad" value="${(entry_outer_diameter - 2*nozzle_wall_width)/2}" />
   <xacro:property name="dist_from_centerline" value="${(throat_middle_diameter + entry_middle_diameter)/4}" />
-  <xacro:property name="slope_angle" value="0.3054949" />
+  <xacro:property name="slope_angle" value="0.3073" />
   <xacro:macro name="nozzle_geom" params="num theta prefix">
     <link name="${prefix}nozzle_geom${num}">

Commit message: hil runner now fully integrated. we are having some issues with sensors getting over torqued but as far as I can tell this is not a software issue and instead will need to be adressed by either opporating closer to the limits or switching sensors.

File: urdf/cv.urdf (robot description, URDF)
Before this commit: robot FREND, 31 links, 30 joints
Joints:
- joint nozzle_to_cone_vertex: origin xyz=0 0 0 rpy=0 0 0 -> xyz=0 0 0.51 rpy=0 0 0

File: urdf/robot_cv_detached.urdf (robot description, URDF)
Before this commit: robot FREND, 48 links, 47 joints
Joints:
- joint nozzle_to_cone_vertex: origin xyz=0 0 0 rpy=0 0 0 -> xyz=0 0 0.51 rpy=0 0 0

File: urdf/simulation/satellite/cv.xacro (robot description, xacro)
@@ -71,5 +71,5 @@
     <parent link="$(arg prefix)nozzle"/>
     <child link="$(arg prefix)cone_vertex"/>
-    <origin rpy="0 0 0" xyz="0 0 0"/>
+    <origin rpy="0 0 0" xyz="0 0 0.51"/>
   </joint>
   <link name="$(arg prefix)hole">
