Commit message: Revert "Holodeck integration/insertion pipeline for demo (#3)"
This reverts commit 2cea9d495a1852177b824da3767f72b207106904.

File: urdf/cv.urdf (robot description, URDF)
Before this commit: robot FREND, 31 links, 30 joints
Links:
- link client: geometry visual mesh filename=package://on_orbit/urdf/simulation/meshes/cv_assembly.stl scale=1 1 1
- link nozzle_geom0: geometry collision box size=0.003 0.04 0.07671
- link nozzle_geom1: geometry collision box size=0.003 0.04 0.07671
- link nozzle_geom2: geometry collision box size=0.003 0.04 0.07671
- link nozzle_geom3: geometry collision box size=0.003 0.04 0.07671
- link nozzle_geom4: geometry collision box size=0.003 0.04 0.07671
- link nozzle_geom5: geometry collision box size=0.003 0.04 0.07671
- link nozzle_geom6: geometry collision box size=0.003 0.04 0.07671
- link nozzle_geom7: geometry collision box size=0.003 0.04 0.07671
Joints:
- joint nozzle_to_capture_box: origin xyz=0 0 -0.05 rpy=0 0 0 -> xyz=0 0 -0.451674428 rpy=0 0 0
- joint nozzle_to_cone_vertex: origin xyz=0 0 0.51 rpy=0 0 0 -> xyz=0 0 0.0748 rpy=0 0 0
- joint nozzle_to_goal: origin xyz=0 0 0.4656 rpy=0 0 0 -> xyz=0 0 0.110 rpy=0 0 0
- joint nozzle_to_hole: origin xyz=0 0 0.429 rpy=0 0 0 -> xyz=0 0 0.0675 rpy=0 0 0
- joint nozzle_to_hole_end: origin xyz=0 0 0.4785 rpy=0 0 0 -> xyz=0 0 0.112 rpy=0 0 0
- joint nozzle_to_nozzle_geom0: origin xyz=0.079 0.0 0.2184025683012885 rpy=0 -0.3073 0 -> xyz=0.029920000000000002 0.0 0.03517396538237974 rpy=0 -0.49514949 0
- joint nozzle_to_nozzle_geom1: origin xyz=0.05586143571373726 0.05586143571373725 0.2184025683012885 rpy=0 -0.3073 0.7853981633974483 -> xyz=0.021156634893101506 0.021156634893101503 0.03517396538237974 rpy=0 -0.49514949 0.7853981633974483
- joint nozzle_to_nozzle_geom2: origin xyz=4.837354856632045e-18 0.079 0.2184025683012885 rpy=0 -0.3073 1.5707963267948966 -> xyz=1.8320716115244406e-18 0.029920000000000002 0.03517396538237974 rpy=0 -0.49514949 1.5707963267948966
- joint nozzle_to_nozzle_geom3: origin xyz=-0.05586143571373725 0.05586143571373726 0.2184025683012885 rpy=0 -0.3073 2.356194490192345 -> xyz=-0.021156634893101503 0.021156634893101506 0.03517396538237974 rpy=0 -0.49514949 2.356194490192345
- joint nozzle_to_nozzle_geom4: origin xyz=-0.079 9.67470971326409e-18 0.2184025683012885 rpy=0 -0.3073 3.141592653589793 -> xyz=-0.029920000000000002 3.664143223048881e-18 0.03517396538237974 rpy=0 -0.49514949 3.141592653589793
- joint nozzle_to_nozzle_geom5: origin xyz=-0.055861435713737265 -0.05586143571373725 0.2184025683012885 rpy=0 -0.3073 3.9269908169872414 -> xyz=-0.021156634893101506 -0.021156634893101503 0.03517396538237974 rpy=0 -0.49514949 3.9269908169872414
- joint nozzle_to_nozzle_geom6: origin xyz=-1.4512064569896134e-17 -0.079 0.2184025683012885 rpy=0 -0.3073 4.71238898038469 -> xyz=-5.496214834573321e-18 -0.029920000000000002 0.03517396538237974 rpy=0 -0.49514949 4.71238898038469
- joint nozzle_to_nozzle_geom7: origin xyz=0.055861435713737244 -0.055861435713737265 0.2184025683012885 rpy=0 -0.3073 5.497787143782138 -> xyz=0.0211566348931015 -0.021156634893101506 0.03517396538237974 rpy=0 -0.49514949 5.497787143782138
- joint nozzle_to_nozzle_rim0: origin xyz=0.142 0.0 0 rpy=0 -0.3073 0 -> xyz=0.04584 0.0 0 rpy=0 -0.49514949 0
- joint nozzle_to_nozzle_rim1: origin xyz=0.10040916292848974 0.10040916292848973 0 rpy=0 -0.3073 0.7853981633974483 -> xyz=0.03241377484959134 0.032413774849591334 0 rpy=0 -0.49514949 0.7853981633974483
- joint nozzle_to_nozzle_rim2: origin xyz=8.694992273946207e-18 0.142 0 rpy=0 -0.3073 1.5707963267948966 -> xyz=2.8068904636457335e-18 0.04584 0 rpy=0 -0.49514949 1.5707963267948966
- joint nozzle_to_nozzle_rim3: origin xyz=-0.10040916292848973 0.10040916292848974 0 rpy=0 -0.3073 2.356194490192345 -> xyz=-0.032413774849591334 0.03241377484959134 0 rpy=0 -0.49514949 2.356194490192345
- joint nozzle_to_nozzle_rim4: origin xyz=-0.142 1.7389984547892414e-17 0 rpy=0 -0.3073 3.141592653589793 -> xyz=-0.04584 5.613780927291467e-18 0 rpy=0 -0.49514949 3.141592653589793
- joint nozzle_to_nozzle_rim5: origin xyz=-0.10040916292848977 -0.10040916292848973 0 rpy=0 -0.3073 3.9269908169872414 -> xyz=-0.03241377484959135 -0.032413774849591334 0 rpy=0 -0.49514949 3.9269908169872414
- joint nozzle_to_nozzle_rim6: origin xyz=-2.6084976821838618e-17 -0.142 0 rpy=0 -0.3073 4.71238898038469 -> xyz=-8.4206713909372e-18 -0.04584 0 rpy=0 -0.49514949 4.71238898038469
- joint nozzle_to_nozzle_rim7: origin xyz=0.10040916292848971 -0.10040916292848977 0 rpy=0 -0.3073 5.497787143782138 -> xyz=0.03241377484959133 -0.03241377484959135 0 rpy=0 -0.49514949 5.497787143782138
- joint nozzle_to_tube_geom0: origin xyz=0.0127 0.0 0.45075 rpy=0 0 0 -> xyz=0.0127 0.0 0.08975 rpy=0 0 0
- joint nozzle_to_tube_geom1: origin xyz=0.008980256121069154 0.008980256121069152 0.45075 rpy=0 0 0.7853981633974483 -> xyz=0.008980256121069154 0.008980256121069152 0.08975 rpy=0 0 0.7853981633974483
- joint nozzle_to_tube_geom2: origin xyz=7.776507174585693e-19 0.0127 0.45075 rpy=0 0 1.5707963267948966 -> xyz=7.776507174585693e-19 0.0127 0.08975 rpy=0 0 1.5707963267948966
- joint nozzle_to_tube_geom3: origin xyz=-0.008980256121069152 0.008980256121069154 0.45075 rpy=0 0 2.356194490192345 -> xyz=-0.008980256121069152 0.008980256121069154 0.08975 rpy=0 0 2.356194490192345
- joint nozzle_to_tube_geom4: origin xyz=-0.0127 1.5553014349171385e-18 0.45075 rpy=0 0 3.141592653589793 -> xyz=-0.0127 1.5553014349171385e-18 0.08975 rpy=0 0 3.141592653589793
- joint nozzle_to_tube_geom5: origin xyz=-0.008980256121069155 -0.008980256121069152 0.45075 rpy=0 0 3.9269908169872414 -> xyz=-0.008980256121069155 -0.008980256121069152 0.08975 rpy=0 0 3.9269908169872414
- joint nozzle_to_tube_geom6: origin xyz=-2.3329521523757078e-18 -0.0127 0.45075 rpy=0 0 4.71238898038469 -> xyz=-2.3329521523757078e-18 -0.0127 0.08975 rpy=0 0 4.71238898038469
- joint nozzle_to_tube_geom7: origin xyz=0.00898025612106915 -0.008980256121069155 0.45075 rpy=0 0 5.497787143782138 -> xyz=0.00898025612106915 -0.008980256121069155 0.08975 rpy=0 0 5.497787143782138

File: urdf/hardware/ur/hw_nozzle_geom.xacro (robot description, xacro)
@@ -1,15 +1,14 @@
 <?xml version="1.0"?>
 <robot xmlns:xacro="http://www.ros.org/wiki/xacro">
-  <xacro:property name="nozzle_length" value="0.4285" />
-  <xacro:property name="nozzle_geom_length" value="0.4551" />
-  <xacro:property name="nozzle_wall_width" value="0.005" />
-  <xacro:property name="nozzle_box_width" value="0.125" />
-  <xacro:property name="throat_outer_diameter" value="0.032" />
+  <xacro:property name="nozzle_length" value="0.0675" />
+  <xacro:property name="nozzle_geom_length" value="0.07671" />
+  <xacro:property name="nozzle_wall_width" value="0.003" />
+  <xacro:property name="nozzle_box_width" value="0.04" />
+  <xacro:property name="throat_outer_diameter" value="0.028" />
   <xacro:property name="throat_middle_diameter" value="${throat_outer_diameter - nozzle_wall_width}" />
-  <xacro:property name="entry_outer_diameter" value="0.294" />
+  <xacro:property name="entry_outer_diameter" value="0.09768" />
   <xacro:property name="entry_middle_diameter" value="${entry_outer_diameter - nozzle_wall_width}" />
-  <xacro:property name="entry_inner_rad" value="${(entry_outer_diameter - 2*nozzle_wall_width)/2}" />
   <xacro:property name="dist_from_centerline" value="${(throat_middle_diameter + entry_middle_diameter)/4}" />
-  <xacro:property name="slope_angle" value="0.3073" />
+  <xacro:property name="slope_angle" value="0.49514949" />
   <xacro:macro name="hw_nozzle_geom" params="num theta">
     <link name="hw_nozzle_geom${num}">

File: urdf/hardware/ur/nozzle_base.xacro (robot description, xacro)
@@ -2,5 +2,5 @@
 <robot xmlns:xacro="http://www.ros.org/wiki/xacro">
   <xacro:property name="nozzle_base_fixture_length" value="0.0095" />
-  <xacro:property name="nozzle_base_fixture_diameter" value="0.063" />
+  <xacro:property name="nozzle_base_fixture_diameter" value="0.06" />
   <xacro:macro name="nozzle_base" params="">
   <link name="nozzle_base">

File: urdf/hardware/ur/ur_3_ur10e.xacro (robot description, xacro)
@@ -3,14 +3,12 @@
   <xacro:include filename="$(find on_orbit)/urdf/hardware/ur/ur10e_macro.xacro"/>
   <xacro:ur10e_robot prefix="ur_3_" calibration_file="$(find on_orbit)/config/holo_params/ur_3_calibration.yaml"/>
-  <xacro:property name="dist_tool_to_ft_sensor" value="0.029" />
-  <!--Peg-->
-  <xacro:property name="peg_rad" value="0.0079"/>
-  <xacro:property name="peg_mass" value="0.260"/>
-  <xacro:property name="peg_com" value="0.071"/>
+  <xacro:property name="dist_tool_to_ft_sensor" value="0.0315" />
+  <!--White Peg-->
   <!-- Will need to be updated after the print-->
-  <!-- Old Value -->
-  <!-- <xacro:property name="ur_3_ee_length" value="0.1558"/> -->
-  <!-- New Value -->
-  <xacro:property name="ur_3_ee_length" value="0.540"/>
+  <xacro:property name="peg_rad" value="0.01505"/>
+  <xacro:property name="peg_mass" value="0.14597807959"/>
+  <xacro:property name="peg_com" value="0.02715593628"/>
+  <!-- Will need to be updated after the print-->
+  <xacro:property name="ur_3_ee_length" value="0.209"/>
   <link name="ur_3_ee">
     <visual>
@@ -46,5 +44,5 @@
     <origin rpy="0 0 0" xyz="0 0 ${ur_3_ee_length}"/>
   </joint>
-  <!-- ur_3 has the FT sensor-->
+  <!-- UR16 has the FT sensor-->
   <link name="ft_sensor"/>
   <joint name="ur_3_tool0_to_ft_sensor" type="fixed">

File: urdf/hardware/ur/ur_4_ur10e.xacro (robot description, xacro)
@@ -6,8 +6,16 @@
   <xacro:include filename="$(find on_orbit)/urdf/hardware/ur/ur10e_macro.xacro"/>
   <xacro:ur10e_robot prefix="ur_4_" calibration_file="$(find on_orbit)/config/holo_params/ur_4_calibration.yaml"/>
+  <xacro:property name="dist_tool_to_ft_sensor" value="0.0315" />
   <!--Short White Nozzle Attached to Robot 4-->
   <!-- Will need to be updated after the print-->
-  <xacro:property name="ur_4_ee_length" value="0.4785"/>
-  <xacro:property name="ur_4_ee_signed_dist_from_ee_to_goal" value="0.4656"/>
+  <xacro:property name="ur_4_ee_length" value="0.12477"/>
+  <xacro:property name="ur_4_ee_signed_dist_from_ee_to_goal" value="0.09017557238"/>
+  <!-- <link name="world"/> -->
+  <!-- <joint name="world_to_ur_4_base_link" type="fixed"> -->
+    <!-- <parent link="world"/> -->
+    <!-- <child link="ur_4_base_link"/> -->
+    <!--We will need to determine true orientation of each of robot as they are at an angle-->
+    <!-- <origin rpy="0 0 0" xyz="0 -0.9948543 -0.00045865"/> -->
+  <!-- </joint> -->
   <link name="hw_goal"/>
   <joint name="ur_4_ee_to_goal" type="fixed">

File: urdf/holodeck.urdf (robot description, URDF)
Before this commit: robot holodeck, 73 links, 72 joints
Links:
- link hw_nozzle_geom0: geometry collision box size=0.003 0.04 0.07671; visual box size=0.003 0.04 0.07671
- link hw_nozzle_geom1: geometry collision box size=0.003 0.04 0.07671; visual box size=0.003 0.04 0.07671
- link hw_nozzle_geom2: geometry collision box size=0.003 0.04 0.07671; visual box size=0.003 0.04 0.07671
- link hw_nozzle_geom3: geometry collision box size=0.003 0.04 0.07671; visual box size=0.003 0.04 0.07671
- link hw_nozzle_geom4: geometry collision box size=0.003 0.04 0.07671; visual box size=0.003 0.04 0.07671
- link hw_nozzle_geom5: geometry collision box size=0.003 0.04 0.07671; visual box size=0.003 0.04 0.07671
- link hw_nozzle_geom6: geometry collision box size=0.003 0.04 0.07671; visual box size=0.003 0.04 0.07671
- link hw_nozzle_geom7: geometry collision box size=0.003 0.04 0.07671; visual box size=0.003 0.04 0.07671
- link nozzle_base: geometry collision cylinder length=0.0095 radius=0.03; visual cylinder length=0.0095 radius=0.03
- link ur_3_ee: mass 0.26 -> 0.14597807959; geometry collision cylinder length=0.209 radius=0.01505; visual cylinder length=0.209 radius=0.01505
Joints:
- joint ur_3_ee_to_peg_center: origin xyz=0 0 -0.27 rpy=0 0 0 -> xyz=0 0 -0.1045 rpy=0 0 0
- joint ur_3_tool0_to_ee: origin xyz=0 0 0.54 rpy=0 0 0 -> xyz=0 0 0.209 rpy=0 0 0
- joint ur_3_tool0_to_ft_sensor: origin xyz=0 0 0.029 rpy=0 0 -0.53996123733 -> xyz=0 0 0.0315 rpy=0 0 -0.53996123733
- joint ur_4_ee_to_goal: origin xyz=0 0 0.4656 rpy=0 3.141592653589793 0 -> xyz=0 0 0.09017557238 rpy=0 3.141592653589793 0
- joint ur_4_ee_to_hw_nozzle_geom0: origin xyz=0.079 0.0 0.2184025683012885 rpy=0 -0.3073 0 -> xyz=0.029920000000000002 0.0 0.03517396538237974 rpy=0 -0.49514949 0
- joint ur_4_ee_to_hw_nozzle_geom1: origin xyz=0.05586143571373726 0.05586143571373725 0.2184025683012885 rpy=0 -0.3073 0.7853981633974483 -> xyz=0.021156634893101506 0.021156634893101503 0.03517396538237974 rpy=0 -0.49514949 0.7853981633974483
- joint ur_4_ee_to_hw_nozzle_geom2: origin xyz=4.837354856632045e-18 0.079 0.2184025683012885 rpy=0 -0.3073 1.5707963267948966 -> xyz=1.8320716115244406e-18 0.029920000000000002 0.03517396538237974 rpy=0 -0.49514949 1.5707963267948966
- joint ur_4_ee_to_hw_nozzle_geom3: origin xyz=-0.05586143571373725 0.05586143571373726 0.2184025683012885 rpy=0 -0.3073 2.356194490192345 -> xyz=-0.021156634893101503 0.021156634893101506 0.03517396538237974 rpy=0 -0.49514949 2.356194490192345
- joint ur_4_ee_to_hw_nozzle_geom4: origin xyz=-0.079 9.67470971326409e-18 0.2184025683012885 rpy=0 -0.3073 3.141592653589793 -> xyz=-0.029920000000000002 3.664143223048881e-18 0.03517396538237974 rpy=0 -0.49514949 3.141592653589793
- joint ur_4_ee_to_hw_nozzle_geom5: origin xyz=-0.055861435713737265 -0.05586143571373725 0.2184025683012885 rpy=0 -0.3073 3.9269908169872414 -> xyz=-0.021156634893101506 -0.021156634893101503 0.03517396538237974 rpy=0 -0.49514949 3.9269908169872414
- joint ur_4_ee_to_hw_nozzle_geom6: origin xyz=-1.4512064569896134e-17 -0.079 0.2184025683012885 rpy=0 -0.3073 4.71238898038469 -> xyz=-5.496214834573321e-18 -0.029920000000000002 0.03517396538237974 rpy=0 -0.49514949 4.71238898038469
- joint ur_4_ee_to_hw_nozzle_geom7: origin xyz=0.055861435713737244 -0.055861435713737265 0.2184025683012885 rpy=0 -0.3073 5.497787143782138 -> xyz=0.0211566348931015 -0.021156634893101506 0.03517396538237974 rpy=0 -0.49514949 5.497787143782138
- joint ur_4_ee_to_tube_geom0: origin xyz=0.0127 0.0 0.45075 rpy=0 0 0 -> xyz=0.0127 0.0 0.08975 rpy=0 0 0
- joint ur_4_ee_to_tube_geom1: origin xyz=0.008980256121069154 0.008980256121069152 0.45075 rpy=0 0 0.7853981633974483 -> xyz=0.008980256121069154 0.008980256121069152 0.08975 rpy=0 0 0.7853981633974483
- joint ur_4_ee_to_tube_geom2: origin xyz=7.776507174585693e-19 0.0127 0.45075 rpy=0 0 1.5707963267948966 -> xyz=7.776507174585693e-19 0.0127 0.08975 rpy=0 0 1.5707963267948966
- joint ur_4_ee_to_tube_geom3: origin xyz=-0.008980256121069152 0.008980256121069154 0.45075 rpy=0 0 2.356194490192345 -> xyz=-0.008980256121069152 0.008980256121069154 0.08975 rpy=0 0 2.356194490192345
- joint ur_4_ee_to_tube_geom4: origin xyz=-0.0127 1.5553014349171385e-18 0.45075 rpy=0 0 3.141592653589793 -> xyz=-0.0127 1.5553014349171385e-18 0.08975 rpy=0 0 3.141592653589793
- joint ur_4_ee_to_tube_geom5: origin xyz=-0.008980256121069155 -0.008980256121069152 0.45075 rpy=0 0 3.9269908169872414 -> xyz=-0.008980256121069155 -0.008980256121069152 0.08975 rpy=0 0 3.9269908169872414
- joint ur_4_ee_to_tube_geom6: origin xyz=-2.3329521523757078e-18 -0.0127 0.45075 rpy=0 0 4.71238898038469 -> xyz=-2.3329521523757078e-18 -0.0127 0.08975 rpy=0 0 4.71238898038469
- joint ur_4_ee_to_tube_geom7: origin xyz=0.00898025612106915 -0.008980256121069155 0.45075 rpy=0 0 5.497787143782138 -> xyz=0.00898025612106915 -0.008980256121069155 0.08975 rpy=0 0 5.497787143782138
- joint ur_4_tool0_to_ee: origin xyz=0 0 0.4785 rpy=0 3.14159 0 -> xyz=0 0 0.12477 rpy=0 3.14159 0

File: urdf/on_orbit_rail.urdf (robot description, URDF)
Before this commit: robot holodeck, 48 links, 47 joints
Links:
- link hw_nozzle_geom0: geometry collision box size=0.003 0.04 0.07671; visual box size=0.003 0.04 0.07671
- link hw_nozzle_geom1: geometry collision box size=0.003 0.04 0.07671; visual box size=0.003 0.04 0.07671
- link hw_nozzle_geom2: geometry collision box size=0.003 0.04 0.07671; visual box size=0.003 0.04 0.07671
- link hw_nozzle_geom3: geometry collision box size=0.003 0.04 0.07671; visual box size=0.003 0.04 0.07671
- link hw_nozzle_geom4: geometry collision box size=0.003 0.04 0.07671; visual box size=0.003 0.04 0.07671
- link hw_nozzle_geom5: geometry collision box size=0.003 0.04 0.07671; visual box size=0.003 0.04 0.07671
- link hw_nozzle_geom6: geometry collision box size=0.003 0.04 0.07671; visual box size=0.003 0.04 0.07671
- link hw_nozzle_geom7: geometry collision box size=0.003 0.04 0.07671; visual box size=0.003 0.04 0.07671
- link nozzle_base: geometry collision cylinder length=0.0095 radius=0.03; visual cylinder length=0.0095 radius=0.03
- link ur_3_ee: mass 0.26 -> 0.14597807959; geometry collision cylinder length=0.209 radius=0.01505; visual cylinder length=0.209 radius=0.01505
Joints:
- joint ur_3_ee_to_peg_center: origin xyz=0 0 -0.27 rpy=0 0 0 -> xyz=0 0 -0.1045 rpy=0 0 0
- joint ur_3_tool0_to_ee: origin xyz=0 0 0.54 rpy=0 0 0 -> xyz=0 0 0.209 rpy=0 0 0
- joint ur_3_tool0_to_ft_sensor: origin xyz=0 0 0.029 rpy=0 0 -0.53996123733 -> xyz=0 0 0.0315 rpy=0 0 -0.53996123733
- joint ur_4_ee_to_goal: origin xyz=0 0 0.4656 rpy=0 3.141592653589793 0 -> xyz=0 0 0.09017557238 rpy=0 3.141592653589793 0
- joint ur_4_ee_to_hw_nozzle_geom0: origin xyz=0.079 0.0 0.2184025683012885 rpy=0 -0.3073 0 -> xyz=0.029920000000000002 0.0 0.03517396538237974 rpy=0 -0.49514949 0
- joint ur_4_ee_to_hw_nozzle_geom1: origin xyz=0.05586143571373726 0.05586143571373725 0.2184025683012885 rpy=0 -0.3073 0.7853981633974483 -> xyz=0.021156634893101506 0.021156634893101503 0.03517396538237974 rpy=0 -0.49514949 0.7853981633974483
- joint ur_4_ee_to_hw_nozzle_geom2: origin xyz=4.837354856632045e-18 0.079 0.2184025683012885 rpy=0 -0.3073 1.5707963267948966 -> xyz=1.8320716115244406e-18 0.029920000000000002 0.03517396538237974 rpy=0 -0.49514949 1.5707963267948966
- joint ur_4_ee_to_hw_nozzle_geom3: origin xyz=-0.05586143571373725 0.05586143571373726 0.2184025683012885 rpy=0 -0.3073 2.356194490192345 -> xyz=-0.021156634893101503 0.021156634893101506 0.03517396538237974 rpy=0 -0.49514949 2.356194490192345
- joint ur_4_ee_to_hw_nozzle_geom4: origin xyz=-0.079 9.67470971326409e-18 0.2184025683012885 rpy=0 -0.3073 3.141592653589793 -> xyz=-0.029920000000000002 3.664143223048881e-18 0.03517396538237974 rpy=0 -0.49514949 3.141592653589793
- joint ur_4_ee_to_hw_nozzle_geom5: origin xyz=-0.055861435713737265 -0.05586143571373725 0.2184025683012885 rpy=0 -0.3073 3.9269908169872414 -> xyz=-0.021156634893101506 -0.021156634893101503 0.03517396538237974 rpy=0 -0.49514949 3.9269908169872414
- joint ur_4_ee_to_hw_nozzle_geom6: origin xyz=-1.4512064569896134e-17 -0.079 0.2184025683012885 rpy=0 -0.3073 4.71238898038469 -> xyz=-5.496214834573321e-18 -0.029920000000000002 0.03517396538237974 rpy=0 -0.49514949 4.71238898038469
- joint ur_4_ee_to_hw_nozzle_geom7: origin xyz=0.055861435713737244 -0.055861435713737265 0.2184025683012885 rpy=0 -0.3073 5.497787143782138 -> xyz=0.0211566348931015 -0.021156634893101506 0.03517396538237974 rpy=0 -0.49514949 5.497787143782138
- joint ur_4_ee_to_tube_geom0: origin xyz=0.0127 0.0 0.45075 rpy=0 0 0 -> xyz=0.0127 0.0 0.08975 rpy=0 0 0
- joint ur_4_ee_to_tube_geom1: origin xyz=0.008980256121069154 0.008980256121069152 0.45075 rpy=0 0 0.7853981633974483 -> xyz=0.008980256121069154 0.008980256121069152 0.08975 rpy=0 0 0.7853981633974483
- joint ur_4_ee_to_tube_geom2: origin xyz=7.776507174585693e-19 0.0127 0.45075 rpy=0 0 1.5707963267948966 -> xyz=7.776507174585693e-19 0.0127 0.08975 rpy=0 0 1.5707963267948966
- joint ur_4_ee_to_tube_geom3: origin xyz=-0.008980256121069152 0.008980256121069154 0.45075 rpy=0 0 2.356194490192345 -> xyz=-0.008980256121069152 0.008980256121069154 0.08975 rpy=0 0 2.356194490192345
- joint ur_4_ee_to_tube_geom4: origin xyz=-0.0127 1.5553014349171385e-18 0.45075 rpy=0 0 3.141592653589793 -> xyz=-0.0127 1.5553014349171385e-18 0.08975 rpy=0 0 3.141592653589793
- joint ur_4_ee_to_tube_geom5: origin xyz=-0.008980256121069155 -0.008980256121069152 0.45075 rpy=0 0 3.9269908169872414 -> xyz=-0.008980256121069155 -0.008980256121069152 0.08975 rpy=0 0 3.9269908169872414
- joint ur_4_ee_to_tube_geom6: origin xyz=-2.3329521523757078e-18 -0.0127 0.45075 rpy=0 0 4.71238898038469 -> xyz=-2.3329521523757078e-18 -0.0127 0.08975 rpy=0 0 4.71238898038469
- joint ur_4_ee_to_tube_geom7: origin xyz=0.00898025612106915 -0.008980256121069155 0.45075 rpy=0 0 5.497787143782138 -> xyz=0.00898025612106915 -0.008980256121069155 0.08975 rpy=0 0 5.497787143782138
- joint ur_4_tool0_to_ee: origin xyz=0 0 0.4785 rpy=0 3.14159 0 -> xyz=0 0 0.12477 rpy=0 3.14159 0

File: urdf/robot.urdf (robot description, URDF)
Before this commit: robot FREND, 16 links, 15 joints
Joints:
- joint ee_peg_joint: origin xyz=0 0 1.3101 rpy=0 0 0 -> xyz=0 0 1.1101 rpy=0 0 0
