Commit message: bug in EKF script had the mass and the inertia of a previous cv model. It has been updated and should improve state estimation.
many plotting scripts have been added that help capture tracking error of the emulator

File: urdf/cv.urdf (robot description, URDF)
Before this commit: robot FREND, 31 links, 30 joints
Links:
- link nozzle_geom0: geometry collision box size=0.005 0.125 0.4551; visual box size=0.005 0.125 0.4551
- link nozzle_geom1: geometry collision box size=0.005 0.125 0.4551; visual box size=0.005 0.125 0.4551
- link nozzle_geom2: geometry collision box size=0.005 0.125 0.4551; visual box size=0.005 0.125 0.4551
- link nozzle_geom3: geometry collision box size=0.005 0.125 0.4551; visual box size=0.005 0.125 0.4551
- link nozzle_geom4: geometry collision box size=0.005 0.125 0.4551; visual box size=0.005 0.125 0.4551
- link nozzle_geom5: geometry collision box size=0.005 0.125 0.4551; visual box size=0.005 0.125 0.4551
- link nozzle_geom6: geometry collision box size=0.005 0.125 0.4551; visual box size=0.005 0.125 0.4551
- link nozzle_geom7: geometry collision box size=0.005 0.125 0.4551; visual box size=0.005 0.125 0.4551

File: urdf/hardware/ur/ur_3_ur10e.xacro (robot description, xacro)
@@ -12,5 +12,5 @@
   <!-- <xacro:property name="ur_3_ee_length" value="0.1558"/> -->
   <!-- New Value -->
-  <xacro:property name="ur_3_ee_length" value="0.5428"/>
+  <xacro:property name="ur_3_ee_length" value="0.547"/>
   <link name="ur_3_ee">
     <visual>

File: urdf/holodeck.urdf (robot description, URDF)
Before this commit: robot holodeck, 73 links, 72 joints
Links:
- link ur_3_ee: geometry collision cylinder length=0.547 radius=0.008; visual cylinder length=0.547 radius=0.008
Joints:
- joint ur_3_ee_to_peg_center: origin xyz=0 0 -0.2714 rpy=0 0 0 -> xyz=0 0 -0.2735 rpy=0 0 0
- joint ur_3_tool0_to_ee: origin xyz=0 0 0.5428 rpy=0 0 0 -> xyz=0 0 0.547 rpy=0 0 0

File: urdf/on_orbit.urdf (robot description, URDF)
Before this commit: robot holodeck, 48 links, 47 joints
Links:
- link ur_3_ee: geometry collision cylinder length=0.547 radius=0.008; visual cylinder length=0.547 radius=0.008
Joints:
- joint ur_3_ee_to_peg_center: origin xyz=0 0 -0.2714 rpy=0 0 0 -> xyz=0 0 -0.2735 rpy=0 0 0
- joint ur_3_tool0_to_ee: origin xyz=0 0 0.5428 rpy=0 0 0 -> xyz=0 0 0.547 rpy=0 0 0

File: urdf/robot_cv_detached.urdf (robot description, URDF)
Before this commit: robot FREND, 48 links, 47 joints
Links:
- link nozzle_geom0: geometry collision box size=0.005 0.125 0.4551; visual box size=0.005 0.125 0.4551
- link nozzle_geom1: geometry collision box size=0.005 0.125 0.4551; visual box size=0.005 0.125 0.4551
- link nozzle_geom2: geometry collision box size=0.005 0.125 0.4551; visual box size=0.005 0.125 0.4551
- link nozzle_geom3: geometry collision box size=0.005 0.125 0.4551; visual box size=0.005 0.125 0.4551
- link nozzle_geom4: geometry collision box size=0.005 0.125 0.4551; visual box size=0.005 0.125 0.4551
- link nozzle_geom5: geometry collision box size=0.005 0.125 0.4551; visual box size=0.005 0.125 0.4551
- link nozzle_geom6: geometry collision box size=0.005 0.125 0.4551; visual box size=0.005 0.125 0.4551
- link nozzle_geom7: geometry collision box size=0.005 0.125 0.4551; visual box size=0.005 0.125 0.4551

File: urdf/simulation/satellite/sim_nozzle_geom.xacro (robot description, xacro)
@@ -14,5 +14,5 @@
   <xacro:macro name="nozzle_geom" params="num theta prefix">
     <link name="${prefix}nozzle_geom${num}">
-      <!-- <visual>
+      <visual>
         <origin rpy="0 0 0" xyz="0 0 0"/>
         <geometry>
@@ -22,5 +22,5 @@
           <color rgba="1.0 1.0 1.0 0.5"/>
         </material>
-      </visual> -->
+      </visual>
       <inertial>
         <mass value="0"/>

File: urdf/single_arm.urdf (robot description, URDF)
Before this commit: robot ur10e_robot, 14 links, 13 joints
Links:
- removed link ft_sensor
- removed link peg_center
- removed link ur_3_base
- removed link ur_3_base_link
- removed link ur_3_base_link_inertia
- removed link ur_3_ee
- removed link ur_3_flange
- removed link ur_3_forearm_link
- removed link ur_3_shoulder_link
- removed link ur_3_tool0
- removed link ur_3_upper_arm_link
- removed link ur_3_wrist_1_link
- removed link ur_3_wrist_2_link
- removed link ur_3_wrist_3_link
- added link ur_1_base
- added link ur_1_base_link
- added link ur_1_base_link_inertia, mass 4.0; collision mesh filename=package://ur_description/meshes/ur10e/collision/base.stl; visual mesh filename=package://ur_description/meshes/ur10e/visual/base.dae
- added link ur_1_flange
- added link ur_1_forearm_link, mass 3.87; collision mesh filename=package://ur_description/meshes/ur10e/collision/forearm.stl; visual mesh filename=package://ur_description/meshes/ur10e/visual/forearm.dae
- added link ur_1_shoulder_link, mass 7.778; collision mesh filename=package://ur_description/meshes/ur10e/collision/shoulder.stl; visual mesh filename=package://ur_description/meshes/ur10e/visual/shoulder.dae
- added link ur_1_tool0
- added link ur_1_upper_arm_link, mass 12.93; collision mesh filename=package://ur_description/meshes/ur10e/collision/upperarm.stl; visual mesh filename=package://ur_description/meshes/ur10e/visual/upperarm.dae
- added link ur_1_wrist_1_link, mass 1.96; collision mesh filename=package://ur_description/meshes/ur10e/collision/wrist1.stl; visual mesh filename=package://ur_description/meshes/ur10e/visual/wrist1.dae
- added link ur_1_wrist_2_link, mass 1.96; collision mesh filename=package://ur_description/meshes/ur10e/collision/wrist2.stl; visual mesh filename=package://ur_description/meshes/ur10e/visual/wrist2.dae
- added link ur_1_wrist_3_link, mass 0.202; collision mesh filename=package://ur_description/meshes/ur10e/collision/wrist3.stl; visual mesh filename=package://ur_description/meshes/ur10e/visual/wrist3.dae
Joints:
- removed joint ur_3_base_link-base_fixed_joint
- removed joint ur_3_base_link-base_link_inertia
- removed joint ur_3_ee_to_peg_center
- removed joint ur_3_elbow_joint
- removed joint ur_3_flange-tool0
- removed joint ur_3_shoulder_lift_joint
- removed joint ur_3_shoulder_pan_joint
- removed joint ur_3_tool0_to_ee
- removed joint ur_3_tool0_to_ft_sensor
- removed joint ur_3_wrist_1_joint
- removed joint ur_3_wrist_2_joint
- removed joint ur_3_wrist_3-flange
- removed joint ur_3_wrist_3_joint
- added joint ur_1_base_link-base_fixed_joint: type fixed, parent ur_1_base_link, child ur_1_base, origin xyz=0 0 0 rpy=0 0 3.141592653589793
- added joint ur_1_base_link-base_link_inertia: type fixed, parent ur_1_base_link, child ur_1_base_link_inertia, origin xyz=0 0 0 rpy=0 0 3.141592653589793
- added joint ur_1_elbow_joint: type revolute, parent ur_1_upper_arm_link, child ur_1_forearm_link, origin xyz=-0.6125449580766956 0 0 rpy=3.140948915487425 3.139929352234192 -3.14159149632371, axis 0 0 1, limit lower=-3.141592653589793 upper=3.141592653589793 effort=150.0 velocity=3.141592653589793
- added joint ur_1_flange-tool0: type fixed, parent ur_1_flange, child ur_1_tool0, origin xyz=0 0 0 rpy=1.5707963267948966 0 1.5707963267948966
- added joint ur_1_shoulder_lift_joint: type revolute, parent ur_1_shoulder_link, child ur_1_upper_arm_link, origin xyz=3.468743937138516e-05 0 0 rpy=1.569800567092754 0 4.521900918381814e-07, axis 0 0 1, limit lower=-6.283185307179586 upper=6.283185307179586 effort=330.0 velocity=2.0943951023931953
- added joint ur_1_shoulder_pan_joint: type revolute, parent ur_1_base_link_inertia, child ur_1_shoulder_link, origin xyz=0 0 0.1808050031292583 rpy=0 0 2.237967734885105e-07, axis 0 0 1, limit lower=-6.283185307179586 upper=6.283185307179586 effort=330.0 velocity=2.0943951023931953
- added joint ur_1_wrist_1_joint: type revolute, parent ur_1_forearm_link, child ur_1_wrist_1_link, origin xyz=-0.5715351569294446 -0.001093047807751683 0.173933352178434 rpy=0.006284208321217083 -0.001639149127442961 5.146417382975639e-06, axis 0 0 1, limit lower=-6.283185307179586 upper=6.283185307179586 effort=56.0 velocity=3.141592653589793
- added joint ur_1_wrist_2_joint: type revolute, parent ur_1_wrist_1_link, child ur_1_wrist_2_link, origin xyz=1.064734108708098e-06 -0.119907694868818 3.734115065993006e-05 rpy=1.570484911005496 0 -7.517950414287489e-08, axis 0 0 1, limit lower=-6.283185307179586 upper=6.283185307179586 effort=56.0 velocity=3.141592653589793
- added joint ur_1_wrist_3-flange: type fixed, parent ur_1_wrist_3_link, child ur_1_flange, origin xyz=0 0 0 rpy=0 -1.5707963267948966 -1.5707963267948966
- added joint ur_1_wrist_3_joint: type revolute, parent ur_1_wrist_2_link, child ur_1_wrist_3_link, origin xyz=-1.372107617229942e-05 0.115539088887634 9.862472815378049e-05 rpy=1.571649931450683 3.141592653589793 -3.141592569298132, axis 0 0 1, limit lower=-6.283185307179586 upper=6.283185307179586 effort=56.0 velocity=3.141592653589793

Commit message: particle filter / ekf comparison and prelimary MPC control working

File: urdf/cv.urdf (robot description, URDF)
Before this commit: robot FREND, 31 links, 30 joints
Links:
- link nozzle_geom0: geometry collision box size=0.005 0.125 0.44712
- link nozzle_geom1: geometry collision box size=0.005 0.125 0.44712
- link nozzle_geom2: geometry collision box size=0.005 0.125 0.44712
- link nozzle_geom3: geometry collision box size=0.005 0.125 0.44712
- link nozzle_geom4: geometry collision box size=0.005 0.125 0.44712
- link nozzle_geom5: geometry collision box size=0.005 0.125 0.44712
- link nozzle_geom6: geometry collision box size=0.005 0.125 0.44712
- link nozzle_geom7: geometry collision box size=0.005 0.125 0.44712
Joints:
- joint nozzle_to_nozzle_geom0: origin xyz=0.079 0.0 0.2184025683012885 rpy=0 -0.3073 0 -> xyz=0.0765 0.0 0.21590863670784355 rpy=0 -0.285672797 0
- joint nozzle_to_nozzle_geom1: origin xyz=0.05586143571373726 0.05586143571373725 0.2184025683012885 rpy=0 -0.3073 0.7853981633974483 -> xyz=0.05409366876077089 0.05409366876077088 0.21590863670784355 rpy=0 -0.285672797 0.7853981633974483
- joint nozzle_to_nozzle_geom2: origin xyz=4.837354856632045e-18 0.079 0.2184025683012885 rpy=0 -0.3073 1.5707963267948966 -> xyz=4.684274006738626e-18 0.0765 0.21590863670784355 rpy=0 -0.285672797 1.5707963267948966
- joint nozzle_to_nozzle_geom3: origin xyz=-0.05586143571373725 0.05586143571373726 0.2184025683012885 rpy=0 -0.3073 2.356194490192345 -> xyz=-0.05409366876077088 0.05409366876077089 0.21590863670784355 rpy=0 -0.285672797 2.356194490192345
- joint nozzle_to_nozzle_geom4: origin xyz=-0.079 9.67470971326409e-18 0.2184025683012885 rpy=0 -0.3073 3.141592653589793 -> xyz=-0.0765 9.368548013477251e-18 0.21590863670784355 rpy=0 -0.285672797 3.141592653589793
- joint nozzle_to_nozzle_geom5: origin xyz=-0.055861435713737265 -0.05586143571373725 0.2184025683012885 rpy=0 -0.3073 3.9269908169872414 -> xyz=-0.054093668760770895 -0.05409366876077088 0.21590863670784355 rpy=0 -0.285672797 3.9269908169872414
- joint nozzle_to_nozzle_geom6: origin xyz=-1.4512064569896134e-17 -0.079 0.2184025683012885 rpy=0 -0.3073 4.71238898038469 -> xyz=-1.4052822020215878e-17 -0.0765 0.21590863670784355 rpy=0 -0.285672797 4.71238898038469
- joint nozzle_to_nozzle_geom7: origin xyz=0.055861435713737244 -0.055861435713737265 0.2184025683012885 rpy=0 -0.3073 5.497787143782138 -> xyz=0.054093668760770874 -0.054093668760770895 0.21590863670784355 rpy=0 -0.285672797 5.497787143782138
- joint nozzle_to_nozzle_rim0: origin xyz=0.142 0.0 0 rpy=0 -0.3073 0 -> xyz=0.13699999999999998 0.0 0 rpy=0 -0.285672797 0
- joint nozzle_to_nozzle_rim1: origin xyz=0.10040916292848974 0.10040916292848973 0 rpy=0 -0.3073 0.7853981633974483 -> xyz=0.096873629022557 0.09687362902255699 0 rpy=0 -0.285672797 0.7853981633974483
- joint nozzle_to_nozzle_rim2: origin xyz=8.694992273946207e-18 0.142 0 rpy=0 -0.3073 1.5707963267948966 -> xyz=8.388830574159368e-18 0.13699999999999998 0 rpy=0 -0.285672797 1.5707963267948966
- joint nozzle_to_nozzle_rim3: origin xyz=-0.10040916292848973 0.10040916292848974 0 rpy=0 -0.3073 2.356194490192345 -> xyz=-0.09687362902255699 0.096873629022557 0 rpy=0 -0.285672797 2.356194490192345
- joint nozzle_to_nozzle_rim4: origin xyz=-0.142 1.7389984547892414e-17 0 rpy=0 -0.3073 3.141592653589793 -> xyz=-0.13699999999999998 1.6777661148318736e-17 0 rpy=0 -0.285672797 3.141592653589793
- joint nozzle_to_nozzle_rim5: origin xyz=-0.10040916292848977 -0.10040916292848973 0 rpy=0 -0.3073 3.9269908169872414 -> xyz=-0.09687362902255701 -0.09687362902255699 0 rpy=0 -0.285672797 3.9269908169872414
- joint nozzle_to_nozzle_rim6: origin xyz=-2.6084976821838618e-17 -0.142 0 rpy=0 -0.3073 4.71238898038469 -> xyz=-2.5166491722478105e-17 -0.13699999999999998 0 rpy=0 -0.285672797 4.71238898038469
- joint nozzle_to_nozzle_rim7: origin xyz=0.10040916292848971 -0.10040916292848977 0 rpy=0 -0.3073 5.497787143782138 -> xyz=0.09687362902255697 -0.09687362902255701 0 rpy=0 -0.285672797 5.497787143782138
- joint nozzle_to_tube_geom0: origin xyz=0.0127 0.0 0.45075 rpy=0 0 0 -> xyz=0.0127 0.0 0.45125 rpy=0 0 0
- joint nozzle_to_tube_geom1: origin xyz=0.008980256121069154 0.008980256121069152 0.45075 rpy=0 0 0.7853981633974483 -> xyz=0.008980256121069154 0.008980256121069152 0.45125 rpy=0 0 0.7853981633974483
- joint nozzle_to_tube_geom2: origin xyz=7.776507174585693e-19 0.0127 0.45075 rpy=0 0 1.5707963267948966 -> xyz=7.776507174585693e-19 0.0127 0.45125 rpy=0 0 1.5707963267948966
- joint nozzle_to_tube_geom3: origin xyz=-0.008980256121069152 0.008980256121069154 0.45075 rpy=0 0 2.356194490192345 -> xyz=-0.008980256121069152 0.008980256121069154 0.45125 rpy=0 0 2.356194490192345
- joint nozzle_to_tube_geom4: origin xyz=-0.0127 1.5553014349171385e-18 0.45075 rpy=0 0 3.141592653589793 -> xyz=-0.0127 1.5553014349171385e-18 0.45125 rpy=0 0 3.141592653589793
- joint nozzle_to_tube_geom5: origin xyz=-0.008980256121069155 -0.008980256121069152 0.45075 rpy=0 0 3.9269908169872414 -> xyz=-0.008980256121069155 -0.008980256121069152 0.45125 rpy=0 0 3.9269908169872414
- joint nozzle_to_tube_geom6: origin xyz=-2.3329521523757078e-18 -0.0127 0.45075 rpy=0 0 4.71238898038469 -> xyz=-2.3329521523757078e-18 -0.0127 0.45125 rpy=0 0 4.71238898038469
- joint nozzle_to_tube_geom7: origin xyz=0.00898025612106915 -0.008980256121069155 0.45075 rpy=0 0 5.497787143782138 -> xyz=0.00898025612106915 -0.008980256121069155 0.45125 rpy=0 0 5.497787143782138

File: urdf/robot_cv_detached.urdf (robot description, URDF)
Before this commit: robot FREND, 48 links, 47 joints
Links:
- link nozzle_geom0: geometry collision box size=0.005 0.125 0.44712
- link nozzle_geom1: geometry collision box size=0.005 0.125 0.44712
- link nozzle_geom2: geometry collision box size=0.005 0.125 0.44712
- link nozzle_geom3: geometry collision box size=0.005 0.125 0.44712
- link nozzle_geom4: geometry collision box size=0.005 0.125 0.44712
- link nozzle_geom5: geometry collision box size=0.005 0.125 0.44712
- link nozzle_geom6: geometry collision box size=0.005 0.125 0.44712
- link nozzle_geom7: geometry collision box size=0.005 0.125 0.44712
Joints:
- joint nozzle_to_nozzle_geom0: origin xyz=0.079 0.0 0.2184025683012885 rpy=0 -0.3073 0 -> xyz=0.0765 0.0 0.21590863670784355 rpy=0 -0.285672797 0
- joint nozzle_to_nozzle_geom1: origin xyz=0.05586143571373726 0.05586143571373725 0.2184025683012885 rpy=0 -0.3073 0.7853981633974483 -> xyz=0.05409366876077089 0.05409366876077088 0.21590863670784355 rpy=0 -0.285672797 0.7853981633974483
- joint nozzle_to_nozzle_geom2: origin xyz=4.837354856632045e-18 0.079 0.2184025683012885 rpy=0 -0.3073 1.5707963267948966 -> xyz=4.684274006738626e-18 0.0765 0.21590863670784355 rpy=0 -0.285672797 1.5707963267948966
- joint nozzle_to_nozzle_geom3: origin xyz=-0.05586143571373725 0.05586143571373726 0.2184025683012885 rpy=0 -0.3073 2.356194490192345 -> xyz=-0.05409366876077088 0.05409366876077089 0.21590863670784355 rpy=0 -0.285672797 2.356194490192345
- joint nozzle_to_nozzle_geom4: origin xyz=-0.079 9.67470971326409e-18 0.2184025683012885 rpy=0 -0.3073 3.141592653589793 -> xyz=-0.0765 9.368548013477251e-18 0.21590863670784355 rpy=0 -0.285672797 3.141592653589793
- joint nozzle_to_nozzle_geom5: origin xyz=-0.055861435713737265 -0.05586143571373725 0.2184025683012885 rpy=0 -0.3073 3.9269908169872414 -> xyz=-0.054093668760770895 -0.05409366876077088 0.21590863670784355 rpy=0 -0.285672797 3.9269908169872414
- joint nozzle_to_nozzle_geom6: origin xyz=-1.4512064569896134e-17 -0.079 0.2184025683012885 rpy=0 -0.3073 4.71238898038469 -> xyz=-1.4052822020215878e-17 -0.0765 0.21590863670784355 rpy=0 -0.285672797 4.71238898038469
- joint nozzle_to_nozzle_geom7: origin xyz=0.055861435713737244 -0.055861435713737265 0.2184025683012885 rpy=0 -0.3073 5.497787143782138 -> xyz=0.054093668760770874 -0.054093668760770895 0.21590863670784355 rpy=0 -0.285672797 5.497787143782138
- joint nozzle_to_nozzle_rim0: origin xyz=0.142 0.0 0 rpy=0 -0.3073 0 -> xyz=0.13699999999999998 0.0 0 rpy=0 -0.285672797 0
- joint nozzle_to_nozzle_rim1: origin xyz=0.10040916292848974 0.10040916292848973 0 rpy=0 -0.3073 0.7853981633974483 -> xyz=0.096873629022557 0.09687362902255699 0 rpy=0 -0.285672797 0.7853981633974483
- joint nozzle_to_nozzle_rim2: origin xyz=8.694992273946207e-18 0.142 0 rpy=0 -0.3073 1.5707963267948966 -> xyz=8.388830574159368e-18 0.13699999999999998 0 rpy=0 -0.285672797 1.5707963267948966
- joint nozzle_to_nozzle_rim3: origin xyz=-0.10040916292848973 0.10040916292848974 0 rpy=0 -0.3073 2.356194490192345 -> xyz=-0.09687362902255699 0.096873629022557 0 rpy=0 -0.285672797 2.356194490192345
- joint nozzle_to_nozzle_rim4: origin xyz=-0.142 1.7389984547892414e-17 0 rpy=0 -0.3073 3.141592653589793 -> xyz=-0.13699999999999998 1.6777661148318736e-17 0 rpy=0 -0.285672797 3.141592653589793
- joint nozzle_to_nozzle_rim5: origin xyz=-0.10040916292848977 -0.10040916292848973 0 rpy=0 -0.3073 3.9269908169872414 -> xyz=-0.09687362902255701 -0.09687362902255699 0 rpy=0 -0.285672797 3.9269908169872414
- joint nozzle_to_nozzle_rim6: origin xyz=-2.6084976821838618e-17 -0.142 0 rpy=0 -0.3073 4.71238898038469 -> xyz=-2.5166491722478105e-17 -0.13699999999999998 0 rpy=0 -0.285672797 4.71238898038469
- joint nozzle_to_nozzle_rim7: origin xyz=0.10040916292848971 -0.10040916292848977 0 rpy=0 -0.3073 5.497787143782138 -> xyz=0.09687362902255697 -0.09687362902255701 0 rpy=0 -0.285672797 5.497787143782138
- joint nozzle_to_tube_geom0: origin xyz=0.0127 0.0 0.45075 rpy=0 0 0 -> xyz=0.0127 0.0 0.45125 rpy=0 0 0
- joint nozzle_to_tube_geom1: origin xyz=0.008980256121069154 0.008980256121069152 0.45075 rpy=0 0 0.7853981633974483 -> xyz=0.008980256121069154 0.008980256121069152 0.45125 rpy=0 0 0.7853981633974483
- joint nozzle_to_tube_geom2: origin xyz=7.776507174585693e-19 0.0127 0.45075 rpy=0 0 1.5707963267948966 -> xyz=7.776507174585693e-19 0.0127 0.45125 rpy=0 0 1.5707963267948966
- joint nozzle_to_tube_geom3: origin xyz=-0.008980256121069152 0.008980256121069154 0.45075 rpy=0 0 2.356194490192345 -> xyz=-0.008980256121069152 0.008980256121069154 0.45125 rpy=0 0 2.356194490192345
- joint nozzle_to_tube_geom4: origin xyz=-0.0127 1.5553014349171385e-18 0.45075 rpy=0 0 3.141592653589793 -> xyz=-0.0127 1.5553014349171385e-18 0.45125 rpy=0 0 3.141592653589793
- joint nozzle_to_tube_geom5: origin xyz=-0.008980256121069155 -0.008980256121069152 0.45075 rpy=0 0 3.9269908169872414 -> xyz=-0.008980256121069155 -0.008980256121069152 0.45125 rpy=0 0 3.9269908169872414
- joint nozzle_to_tube_geom6: origin xyz=-2.3329521523757078e-18 -0.0127 0.45075 rpy=0 0 4.71238898038469 -> xyz=-2.3329521523757078e-18 -0.0127 0.45125 rpy=0 0 4.71238898038469
- joint nozzle_to_tube_geom7: origin xyz=0.00898025612106915 -0.008980256121069155 0.45075 rpy=0 0 5.497787143782138 -> xyz=0.00898025612106915 -0.008980256121069155 0.45125 rpy=0 0 5.497787143782138

File: urdf/simulation/satellite/sim_nozzle_geom.xacro (robot description, xacro)
@@ -1,18 +1,18 @@
 <?xml version="1.0"?>
 <robot xmlns:xacro="http://www.ros.org/wiki/xacro">
-  <xacro:property name="nozzle_length" value="0.4285" />
-  <xacro:property name="nozzle_geom_length" value="0.4551" />
+  <xacro:property name="nozzle_length" value="0.429" />
+  <xacro:property name="nozzle_geom_length" value="0.44712" />
   <xacro:property name="nozzle_wall_width" value="0.005" />
   <xacro:property name="nozzle_box_width" value="0.125" />
   <xacro:property name="throat_outer_diameter" value="0.032" />
   <xacro:property name="throat_middle_diameter" value="${throat_outer_diameter - nozzle_wall_width}" />
-  <xacro:property name="entry_outer_diameter" value="0.294" />
+  <xacro:property name="entry_outer_diameter" value="0.284" />
   <xacro:property name="entry_middle_diameter" value="${entry_outer_diameter - nozzle_wall_width}" />
   <xacro:property name="entry_inner_rad" value="${(entry_outer_diameter - 2*nozzle_wall_width)/2}" />
   <xacro:property name="dist_from_centerline" value="${(throat_middle_diameter + entry_middle_diameter)/4}" />
-  <xacro:property name="slope_angle" value="0.3073" />
+  <xacro:property name="slope_angle" value="0.285672797" />
   <xacro:macro name="nozzle_geom" params="num theta prefix">
     <link name="${prefix}nozzle_geom${num}">
-      <visual>
+      <!-- <visual>
         <origin rpy="0 0 0" xyz="0 0 0"/>
         <geometry>
@@ -22,5 +22,5 @@
           <color rgba="1.0 1.0 1.0 0.5"/>
         </material>
-      </visual>
+      </visual> -->
       <inertial>
         <mass value="0"/>

Commit message: TV-LQR working. New plots created. this branch should be merged into main

File: urdf/cv.urdf (robot description, URDF)
Before this commit: robot FREND, 31 links, 30 joints
Joints:
- joint nozzle_to_capture_box: origin xyz=0 0 -0.07 rpy=0 0 0 -> xyz=0 0 -0.05 rpy=0 0 0

File: urdf/robot_cv_detached.urdf (robot description, URDF)
Before this commit: robot FREND, 48 links, 47 joints
Joints:
- joint nozzle_to_capture_box: origin xyz=0 0 -0.07 rpy=0 0 0 -> xyz=0 0 -0.05 rpy=0 0 0
