Commit message: Holodeck integration/planning (#7)
Preliminary TV-LQR and MPC added

File: urdf/cv.urdf (robot description, URDF)
Before this commit: robot FREND, 31 links, 30 joints
Links:
- link nozzle_geom0: geometry collision box size=0.005 0.125 0.44712
- link nozzle_geom1: geometry collision box size=0.005 0.125 0.44712
- link nozzle_geom2: geometry collision box size=0.005 0.125 0.44712
- link nozzle_geom3: geometry collision box size=0.005 0.125 0.44712
- link nozzle_geom4: geometry collision box size=0.005 0.125 0.44712
- link nozzle_geom5: geometry collision box size=0.005 0.125 0.44712
- link nozzle_geom6: geometry collision box size=0.005 0.125 0.44712
- link nozzle_geom7: geometry collision box size=0.005 0.125 0.44712
Joints:
- joint nozzle_to_nozzle_geom0: origin xyz=0.079 0.0 0.2184025683012885 rpy=0 -0.3073 0 -> xyz=0.0765 0.0 0.21590863670784355 rpy=0 -0.285672797 0
- joint nozzle_to_nozzle_geom1: origin xyz=0.05586143571373726 0.05586143571373725 0.2184025683012885 rpy=0 -0.3073 0.7853981633974483 -> xyz=0.05409366876077089 0.05409366876077088 0.21590863670784355 rpy=0 -0.285672797 0.7853981633974483
- joint nozzle_to_nozzle_geom2: origin xyz=4.837354856632045e-18 0.079 0.2184025683012885 rpy=0 -0.3073 1.5707963267948966 -> xyz=4.684274006738626e-18 0.0765 0.21590863670784355 rpy=0 -0.285672797 1.5707963267948966
- joint nozzle_to_nozzle_geom3: origin xyz=-0.05586143571373725 0.05586143571373726 0.2184025683012885 rpy=0 -0.3073 2.356194490192345 -> xyz=-0.05409366876077088 0.05409366876077089 0.21590863670784355 rpy=0 -0.285672797 2.356194490192345
- joint nozzle_to_nozzle_geom4: origin xyz=-0.079 9.67470971326409e-18 0.2184025683012885 rpy=0 -0.3073 3.141592653589793 -> xyz=-0.0765 9.368548013477251e-18 0.21590863670784355 rpy=0 -0.285672797 3.141592653589793
- joint nozzle_to_nozzle_geom5: origin xyz=-0.055861435713737265 -0.05586143571373725 0.2184025683012885 rpy=0 -0.3073 3.9269908169872414 -> xyz=-0.054093668760770895 -0.05409366876077088 0.21590863670784355 rpy=0 -0.285672797 3.9269908169872414
- joint nozzle_to_nozzle_geom6: origin xyz=-1.4512064569896134e-17 -0.079 0.2184025683012885 rpy=0 -0.3073 4.71238898038469 -> xyz=-1.4052822020215878e-17 -0.0765 0.21590863670784355 rpy=0 -0.285672797 4.71238898038469
- joint nozzle_to_nozzle_geom7: origin xyz=0.055861435713737244 -0.055861435713737265 0.2184025683012885 rpy=0 -0.3073 5.497787143782138 -> xyz=0.054093668760770874 -0.054093668760770895 0.21590863670784355 rpy=0 -0.285672797 5.497787143782138
- joint nozzle_to_nozzle_rim0: origin xyz=0.142 0.0 0 rpy=0 -0.3073 0 -> xyz=0.13699999999999998 0.0 0 rpy=0 -0.285672797 0
- joint nozzle_to_nozzle_rim1: origin xyz=0.10040916292848974 0.10040916292848973 0 rpy=0 -0.3073 0.7853981633974483 -> xyz=0.096873629022557 0.09687362902255699 0 rpy=0 -0.285672797 0.7853981633974483
- joint nozzle_to_nozzle_rim2: origin xyz=8.694992273946207e-18 0.142 0 rpy=0 -0.3073 1.5707963267948966 -> xyz=8.388830574159368e-18 0.13699999999999998 0 rpy=0 -0.285672797 1.5707963267948966
- joint nozzle_to_nozzle_rim3: origin xyz=-0.10040916292848973 0.10040916292848974 0 rpy=0 -0.3073 2.356194490192345 -> xyz=-0.09687362902255699 0.096873629022557 0 rpy=0 -0.285672797 2.356194490192345
- joint nozzle_to_nozzle_rim4: origin xyz=-0.142 1.7389984547892414e-17 0 rpy=0 -0.3073 3.141592653589793 -> xyz=-0.13699999999999998 1.6777661148318736e-17 0 rpy=0 -0.285672797 3.141592653589793
- joint nozzle_to_nozzle_rim5: origin xyz=-0.10040916292848977 -0.10040916292848973 0 rpy=0 -0.3073 3.9269908169872414 -> xyz=-0.09687362902255701 -0.09687362902255699 0 rpy=0 -0.285672797 3.9269908169872414
- joint nozzle_to_nozzle_rim6: origin xyz=-2.6084976821838618e-17 -0.142 0 rpy=0 -0.3073 4.71238898038469 -> xyz=-2.5166491722478105e-17 -0.13699999999999998 0 rpy=0 -0.285672797 4.71238898038469
- joint nozzle_to_nozzle_rim7: origin xyz=0.10040916292848971 -0.10040916292848977 0 rpy=0 -0.3073 5.497787143782138 -> xyz=0.09687362902255697 -0.09687362902255701 0 rpy=0 -0.285672797 5.497787143782138
- joint nozzle_to_tube_geom0: origin xyz=0.0127 0.0 0.45075 rpy=0 0 0 -> xyz=0.0127 0.0 0.45125 rpy=0 0 0
- joint nozzle_to_tube_geom1: origin xyz=0.008980256121069154 0.008980256121069152 0.45075 rpy=0 0 0.7853981633974483 -> xyz=0.008980256121069154 0.008980256121069152 0.45125 rpy=0 0 0.7853981633974483
- joint nozzle_to_tube_geom2: origin xyz=7.776507174585693e-19 0.0127 0.45075 rpy=0 0 1.5707963267948966 -> xyz=7.776507174585693e-19 0.0127 0.45125 rpy=0 0 1.5707963267948966
- joint nozzle_to_tube_geom3: origin xyz=-0.008980256121069152 0.008980256121069154 0.45075 rpy=0 0 2.356194490192345 -> xyz=-0.008980256121069152 0.008980256121069154 0.45125 rpy=0 0 2.356194490192345
- joint nozzle_to_tube_geom4: origin xyz=-0.0127 1.5553014349171385e-18 0.45075 rpy=0 0 3.141592653589793 -> xyz=-0.0127 1.5553014349171385e-18 0.45125 rpy=0 0 3.141592653589793
- joint nozzle_to_tube_geom5: origin xyz=-0.008980256121069155 -0.008980256121069152 0.45075 rpy=0 0 3.9269908169872414 -> xyz=-0.008980256121069155 -0.008980256121069152 0.45125 rpy=0 0 3.9269908169872414
- joint nozzle_to_tube_geom6: origin xyz=-2.3329521523757078e-18 -0.0127 0.45075 rpy=0 0 4.71238898038469 -> xyz=-2.3329521523757078e-18 -0.0127 0.45125 rpy=0 0 4.71238898038469
- joint nozzle_to_tube_geom7: origin xyz=0.00898025612106915 -0.008980256121069155 0.45075 rpy=0 0 5.497787143782138 -> xyz=0.00898025612106915 -0.008980256121069155 0.45125 rpy=0 0 5.497787143782138

File: urdf/hardware/ur/ur_3_ur10e.xacro (robot description, xacro)
@@ -4,5 +4,9 @@
   <xacro:ur10e_robot prefix="ur_3_" calibration_file="$(find on_orbit)/config/holo_params/ur_3_calibration.yaml"/>
   <xacro:property name="dist_tool_to_ft_sensor" value="0.03175" />
+  <xacro:property name="dist_tool_to_ft_sensor" value="0.03175" />
   <!--Peg-->
+  <xacro:property name="peg_rad" value="0.008"/>
+  <xacro:property name="peg_mass" value="0.130"/>
+  <xacro:property name="peg_com" value="0.125"/>
   <xacro:property name="peg_rad" value="0.008"/>
   <xacro:property name="peg_mass" value="0.130"/>
@@ -12,5 +16,5 @@
   <!-- <xacro:property name="ur_3_ee_length" value="0.1558"/> -->
   <!-- New Value -->
-  <xacro:property name="ur_3_ee_length" value="0.5428"/>
+  <xacro:property name="ur_3_ee_length" value="0.547"/>
   <link name="ur_3_ee">
     <visual>

File: urdf/holodeck.urdf (robot description, URDF)
Before this commit: robot holodeck, 73 links, 72 joints
Links:
- link ur_3_ee: geometry collision cylinder length=0.547 radius=0.008; visual cylinder length=0.547 radius=0.008
Joints:
- joint ur_3_ee_to_peg_center: origin xyz=0 0 -0.2714 rpy=0 0 0 -> xyz=0 0 -0.2735 rpy=0 0 0
- joint ur_3_tool0_to_ee: origin xyz=0 0 0.5428 rpy=0 0 0 -> xyz=0 0 0.547 rpy=0 0 0

File: urdf/mrv_ur_arm.urdf (robot description, URDF)
Before this commit: robot ur10e_robot, 14 links, 13 joints
Links:
- link ur_3_ee: geometry collision cylinder length=0.547 radius=0.008; visual cylinder length=0.547 radius=0.008
Joints:
- joint ur_3_ee_to_peg_center: origin xyz=0 0 -0.2714 rpy=0 0 0 -> xyz=0 0 -0.2735 rpy=0 0 0
- joint ur_3_tool0_to_ee: origin xyz=0 0 0.5428 rpy=0 0 0 -> xyz=0 0 0.547 rpy=0 0 0

File: urdf/on_orbit.urdf (robot description, URDF)
Before this commit: robot holodeck, 48 links, 47 joints
Links:
- link ur_3_ee: geometry collision cylinder length=0.547 radius=0.008; visual cylinder length=0.547 radius=0.008
Joints:
- joint ur_3_ee_to_peg_center: origin xyz=0 0 -0.2714 rpy=0 0 0 -> xyz=0 0 -0.2735 rpy=0 0 0
- joint ur_3_tool0_to_ee: origin xyz=0 0 0.5428 rpy=0 0 0 -> xyz=0 0 0.547 rpy=0 0 0

File: urdf/robot_cv_detached.urdf (robot description, URDF)
Before this commit: robot FREND, 48 links, 47 joints
Links:
- link nozzle_geom0: geometry collision box size=0.005 0.125 0.44712
- link nozzle_geom1: geometry collision box size=0.005 0.125 0.44712
- link nozzle_geom2: geometry collision box size=0.005 0.125 0.44712
- link nozzle_geom3: geometry collision box size=0.005 0.125 0.44712
- link nozzle_geom4: geometry collision box size=0.005 0.125 0.44712
- link nozzle_geom5: geometry collision box size=0.005 0.125 0.44712
- link nozzle_geom6: geometry collision box size=0.005 0.125 0.44712
- link nozzle_geom7: geometry collision box size=0.005 0.125 0.44712
Joints:
- joint nozzle_to_nozzle_geom0: origin xyz=0.079 0.0 0.2184025683012885 rpy=0 -0.3073 0 -> xyz=0.0765 0.0 0.21590863670784355 rpy=0 -0.285672797 0
- joint nozzle_to_nozzle_geom1: origin xyz=0.05586143571373726 0.05586143571373725 0.2184025683012885 rpy=0 -0.3073 0.7853981633974483 -> xyz=0.05409366876077089 0.05409366876077088 0.21590863670784355 rpy=0 -0.285672797 0.7853981633974483
- joint nozzle_to_nozzle_geom2: origin xyz=4.837354856632045e-18 0.079 0.2184025683012885 rpy=0 -0.3073 1.5707963267948966 -> xyz=4.684274006738626e-18 0.0765 0.21590863670784355 rpy=0 -0.285672797 1.5707963267948966
- joint nozzle_to_nozzle_geom3: origin xyz=-0.05586143571373725 0.05586143571373726 0.2184025683012885 rpy=0 -0.3073 2.356194490192345 -> xyz=-0.05409366876077088 0.05409366876077089 0.21590863670784355 rpy=0 -0.285672797 2.356194490192345
- joint nozzle_to_nozzle_geom4: origin xyz=-0.079 9.67470971326409e-18 0.2184025683012885 rpy=0 -0.3073 3.141592653589793 -> xyz=-0.0765 9.368548013477251e-18 0.21590863670784355 rpy=0 -0.285672797 3.141592653589793
- joint nozzle_to_nozzle_geom5: origin xyz=-0.055861435713737265 -0.05586143571373725 0.2184025683012885 rpy=0 -0.3073 3.9269908169872414 -> xyz=-0.054093668760770895 -0.05409366876077088 0.21590863670784355 rpy=0 -0.285672797 3.9269908169872414
- joint nozzle_to_nozzle_geom6: origin xyz=-1.4512064569896134e-17 -0.079 0.2184025683012885 rpy=0 -0.3073 4.71238898038469 -> xyz=-1.4052822020215878e-17 -0.0765 0.21590863670784355 rpy=0 -0.285672797 4.71238898038469
- joint nozzle_to_nozzle_geom7: origin xyz=0.055861435713737244 -0.055861435713737265 0.2184025683012885 rpy=0 -0.3073 5.497787143782138 -> xyz=0.054093668760770874 -0.054093668760770895 0.21590863670784355 rpy=0 -0.285672797 5.497787143782138
- joint nozzle_to_nozzle_rim0: origin xyz=0.142 0.0 0 rpy=0 -0.3073 0 -> xyz=0.13699999999999998 0.0 0 rpy=0 -0.285672797 0
- joint nozzle_to_nozzle_rim1: origin xyz=0.10040916292848974 0.10040916292848973 0 rpy=0 -0.3073 0.7853981633974483 -> xyz=0.096873629022557 0.09687362902255699 0 rpy=0 -0.285672797 0.7853981633974483
- joint nozzle_to_nozzle_rim2: origin xyz=8.694992273946207e-18 0.142 0 rpy=0 -0.3073 1.5707963267948966 -> xyz=8.388830574159368e-18 0.13699999999999998 0 rpy=0 -0.285672797 1.5707963267948966
- joint nozzle_to_nozzle_rim3: origin xyz=-0.10040916292848973 0.10040916292848974 0 rpy=0 -0.3073 2.356194490192345 -> xyz=-0.09687362902255699 0.096873629022557 0 rpy=0 -0.285672797 2.356194490192345
- joint nozzle_to_nozzle_rim4: origin xyz=-0.142 1.7389984547892414e-17 0 rpy=0 -0.3073 3.141592653589793 -> xyz=-0.13699999999999998 1.6777661148318736e-17 0 rpy=0 -0.285672797 3.141592653589793
- joint nozzle_to_nozzle_rim5: origin xyz=-0.10040916292848977 -0.10040916292848973 0 rpy=0 -0.3073 3.9269908169872414 -> xyz=-0.09687362902255701 -0.09687362902255699 0 rpy=0 -0.285672797 3.9269908169872414
- joint nozzle_to_nozzle_rim6: origin xyz=-2.6084976821838618e-17 -0.142 0 rpy=0 -0.3073 4.71238898038469 -> xyz=-2.5166491722478105e-17 -0.13699999999999998 0 rpy=0 -0.285672797 4.71238898038469
- joint nozzle_to_nozzle_rim7: origin xyz=0.10040916292848971 -0.10040916292848977 0 rpy=0 -0.3073 5.497787143782138 -> xyz=0.09687362902255697 -0.09687362902255701 0 rpy=0 -0.285672797 5.497787143782138
- joint nozzle_to_tube_geom0: origin xyz=0.0127 0.0 0.45075 rpy=0 0 0 -> xyz=0.0127 0.0 0.45125 rpy=0 0 0
- joint nozzle_to_tube_geom1: origin xyz=0.008980256121069154 0.008980256121069152 0.45075 rpy=0 0 0.7853981633974483 -> xyz=0.008980256121069154 0.008980256121069152 0.45125 rpy=0 0 0.7853981633974483
- joint nozzle_to_tube_geom2: origin xyz=7.776507174585693e-19 0.0127 0.45075 rpy=0 0 1.5707963267948966 -> xyz=7.776507174585693e-19 0.0127 0.45125 rpy=0 0 1.5707963267948966
- joint nozzle_to_tube_geom3: origin xyz=-0.008980256121069152 0.008980256121069154 0.45075 rpy=0 0 2.356194490192345 -> xyz=-0.008980256121069152 0.008980256121069154 0.45125 rpy=0 0 2.356194490192345
- joint nozzle_to_tube_geom4: origin xyz=-0.0127 1.5553014349171385e-18 0.45075 rpy=0 0 3.141592653589793 -> xyz=-0.0127 1.5553014349171385e-18 0.45125 rpy=0 0 3.141592653589793
- joint nozzle_to_tube_geom5: origin xyz=-0.008980256121069155 -0.008980256121069152 0.45075 rpy=0 0 3.9269908169872414 -> xyz=-0.008980256121069155 -0.008980256121069152 0.45125 rpy=0 0 3.9269908169872414
- joint nozzle_to_tube_geom6: origin xyz=-2.3329521523757078e-18 -0.0127 0.45075 rpy=0 0 4.71238898038469 -> xyz=-2.3329521523757078e-18 -0.0127 0.45125 rpy=0 0 4.71238898038469
- joint nozzle_to_tube_geom7: origin xyz=0.00898025612106915 -0.008980256121069155 0.45075 rpy=0 0 5.497787143782138 -> xyz=0.00898025612106915 -0.008980256121069155 0.45125 rpy=0 0 5.497787143782138

File: urdf/simulation/satellite/sim_nozzle_geom.xacro (robot description, xacro)
@@ -1,15 +1,15 @@
 <?xml version="1.0"?>
 <robot xmlns:xacro="http://www.ros.org/wiki/xacro">
-  <xacro:property name="nozzle_length" value="0.4285" />
-  <xacro:property name="nozzle_geom_length" value="0.4551" />
+  <xacro:property name="nozzle_length" value="0.429" />
+  <xacro:property name="nozzle_geom_length" value="0.44712" />
   <xacro:property name="nozzle_wall_width" value="0.005" />
   <xacro:property name="nozzle_box_width" value="0.125" />
   <xacro:property name="throat_outer_diameter" value="0.032" />
   <xacro:property name="throat_middle_diameter" value="${throat_outer_diameter - nozzle_wall_width}" />
-  <xacro:property name="entry_outer_diameter" value="0.294" />
+  <xacro:property name="entry_outer_diameter" value="0.284" />
   <xacro:property name="entry_middle_diameter" value="${entry_outer_diameter - nozzle_wall_width}" />
   <xacro:property name="entry_inner_rad" value="${(entry_outer_diameter - 2*nozzle_wall_width)/2}" />
   <xacro:property name="dist_from_centerline" value="${(throat_middle_diameter + entry_middle_diameter)/4}" />
-  <xacro:property name="slope_angle" value="0.3073" />
+  <xacro:property name="slope_angle" value="0.285672797" />
   <xacro:macro name="nozzle_geom" params="num theta prefix">
     <link name="${prefix}nozzle_geom${num}">
