Commit message: commit before demo 12/2/24

File: urdf/robot_cv_detached.urdf (robot description, URDF)
Before this commit: robot FREND, 48 links, 47 joints
Joints:
- joint joint0: origin xyz=0.3182 -0.3182 1.9875 rpy=0 0 1.047196667 -> xyz=-0.3182 0.3182 1.9875 rpy=0 0 -2.0969

File: urdf/simulation/satellite/robot_cv_detached.xacro (robot description, xacro)
@@ -18,4 +18,5 @@
     <parent link="world"/>
     <child link="$(arg prefix)base_link"/>
+    <!-- <origin rpy="0 0 3.14159" xyz="0 0 0"/> -->
   </joint>
 </robot>
