Commit message: read me updated (good start may need editing)

File: urdf/robot.urdf (robot description, URDF)
Before this commit: robot FREND, 16 links, 15 joints
Joints:
- joint joint0: origin xyz=0.3182 -0.3182 1.9875 rpy=0 0 1.047196667 -> xyz=-0.3182 0.3182 1.9875 rpy=0 0 -2.0969

File: urdf/simulation/satellite/robot.xacro (robot description, xacro)
@@ -37,5 +37,6 @@
   <parent link="$(arg prefix)base_link"/>
     <child link="$(arg prefix)link0"/>
-    <origin rpy="0 0 1.047196667" xyz="0.3182 -0.3182 1.9875"/>
+    <!-- <origin rpy="0 0 1.047196667" xyz="0.3182 -0.3182 1.9875"/> -->
+    <origin rpy="0 0 -2.0969" xyz="-0.3182 0.3182 1.9875"/>
   </joint>
   <link name="$(arg prefix)link0">
