Commit message: add collision geometry for CV

File: urdf/simulation/satellite/cv.xacro (robot description, xacro)
@@ -18,4 +18,10 @@
       </material>
     </visual>
+    <collision>
+    <origin rpy="0 0 0" xyz="0 0 0"/>
+      <geometry>
+        <mesh filename="package://on_orbit/urdf/meshes/full_cv.stl" scale="1 1 1"/>
+      </geometry>
+    </collision>
     <inertial>
       <mass value="${1050*mass_scale}"/>
