Commit message: add cv and MRV w two arms xacro

File: urdf/simulation/satellite/MRV_w_two_arms.xacro (robot description, xacro)
@@ -30,4 +30,9 @@
     </collision>
   </link>
+  <link name="solar_panel_right">
+    <visual>
+    <origin rpy="0 0 0" xyz="2.068/2+2.328+12.405/2 0 3.975/2-2.41"/>
+    </visual>
+  </link>
 <!--Primary Arm-->
 <xacro:frend_arm prefix="primary_"/>
